File: hardware/6502sbc/DMA_cpu_board_interface.kicad_sch (KiCad schematic)
At the start: 15 parts, among them J20 DATA, ADDR, J21 DMA_CTRL, J22 DMA_CTRL, J23 DATA, ADDR, U2 SN74LS07, U25 74AHC2G32DP, U36 74AHC2G32DP

Commit message: Preliminary schematic
Parts:
- renumbered J21 to J22, J22 to J23, J20 to J24, J23 to J25, JP15 to JP21, R27 to R28, TP6 to TP4, TP3 to TP6, TP4 to TP7, U36 to U10, U2 to U5, U25 to U8
Changed lines of the file:
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@@
 		(dnp no)
 		(fields_autoplaced yes)
-		(property "Reference" "U36"
+		(property "Reference" "U10"
 			(at 90.17 52.07 0)
 			(effects
@@
 			(project "6502sbc"
 				(path "/dc8636f6-e59e-4c75-ae27-408ad57a23de/5a0be038-7c3c-4556-9482-35a902da59e6"
-					(reference "U36")
+					(reference "U10")
 					(unit 2)
 				)
@@
 		(dnp no)
 		(fields_autoplaced yes)
-		(property "Reference" "U25"
+		(property "Reference" "U8"
 			(at 63.5 132.0799 90)
 			(effects
@@
 			(project ""
 				(path "/dc8636f6-e59e-4c75-ae27-408ad57a23de/5a0be038-7c3c-4556-9482-35a902da59e6"
-					(reference "U25")
+					(reference "U8")
 					(unit 1)
 				)
@@
 		(on_board yes)
 		(dnp no)
-		(property "Reference" "TP4"
+		(property "Reference" "TP7"
 			(at 140.462 66.294 90)
 			(effects
@@
 			(project ""
 				(path "/dc8636f6-e59e-4c75-ae27-408ad57a23de/5a0be038-7c3c-4556-9482-35a902da59e6"
-					(reference "TP4")
+					(reference "TP7")
 					(unit 1)
 				)
@@
 		(dnp no)
 		(fields_autoplaced yes)
-		(property "Reference" "#PWR0103"
+		(property "Reference" "#PWR0102"
 			(at 215.9 119.38 0)
 			(effects
@@
 			(project "6502sbc"
 				(path "/dc8636f6-e59e-4c75-ae27-408ad57a23de/5a0be038-7c3c-4556-9482-35a902da59e6"
-					(reference "#PWR0103")
+					(reference "#PWR0102")
 					(unit 1)
 				)
@@
 		(dnp no)
 		(fields_autoplaced yes)
-		(property "Reference" "#PWR0105"
+		(property "Reference" "#PWR0104"
 			(at 223.52 129.54 0)
 			(effects
@@
 			(project "6502sbc"
 				(path "/dc8636f6-e59e-4c75-ae27-408ad57a23de/5a0be038-7c3c-4556-9482-35a902da59e6"
-					(reference "#PWR0105")
+					(reference "#PWR0104")
 					(unit 1)
 				)
@@
 		(dnp no)
 		(fields_autoplaced yes)
-		(property "Reference" "U25"
+		(property "Reference" "U8"
 			(at 113.03 102.87 0)
 			(effects
@@
 			(project "6502sbc"
 				(path "/dc8636f6-e59e-4c75-ae27-408ad57a23de/5a0be038-7c3c-4556-9482-35a902da59e6"
-					(reference "U25")
+					(reference "U8")
 					(unit 2)
 				)
@@
 		(dnp no)
 		(fields_autoplaced yes)
-		(property "Reference" "#PWR0108"
+		(property "Reference" "#PWR099"
 			(at 121.92 144.78 0)
 			(effects
@@
 			(project "6502sbc"
 				(path "/dc8636f6-e59e-4c75-ae27-408ad57a23de/5a0be038-7c3c-4556-9482-35a902da59e6"
-					(reference "#PWR0108")
+					(reference "#PWR099")
 					(unit 1)
 				)
@@
 		(dnp no)
 		(fields_autoplaced yes)
-		(property "Reference" "#PWR0100"
+		(property "Reference" "#PWR0108"
 			(at 267.97 64.77 0)
 			(effects
@@
 			(project ""
 				(path "/dc8636f6-e59e-4c75-ae27-408ad57a23de/5a0be038-7c3c-4556-9482-35a902da59e6"
-					(reference "#PWR0100")
+					(reference "#PWR0108")
 					(unit 1)
 				)
@@
 		(dnp no)
 		(fields_autoplaced yes)
-		(property "Reference" "#PWR0102"
+		(property "Reference" "#PWR0101"
 			(at 186.69 119.38 0)
 			(effects
@@
 			(project "6502sbc"
 				(path "/dc8636f6-e59e-4c75-ae27-408ad57a23de/5a0be038-7c3c-4556-9482-35a902da59e6"
-					(reference "#PWR0102")
+					(reference "#PWR0101")
 					(unit 1)
 				)
@@
 		(dnp no)
 		(fields_autoplaced yes)
-		(property "Reference" "J20"
+		(property "Reference" "J24"
 			(at 201.93 114.3 0)
 			(effects
@@
 			(project "6502sbc"
 				(path "/dc8636f6-e59e-4c75-ae27-408ad57a23de/5a0be038-7c3c-4556-9482-35a902da59e6"
-					(reference "J20")
+					(reference "J24")
 					(unit 1)
 				)
@@
 		(dnp no)
 		(fields_autoplaced yes)
-		(property "Reference" "#PWR089"
+		(property "Reference" "#PWR0105"
 			(at 231.14 54.61 0)
 			(effects
@@
 			(project ""
 				(path "/dc8636f6-e59e-4c75-ae27-408ad57a23de/5a0be038-7c3c-4556-9482-35a902da59e6"
-					(reference "#PWR089")
+					(reference "#PWR0105")
 					(unit 1)
 				)
@@
 		(on_board yes)
 		(dnp no)
-		(property "Reference" "J21"
+		(property "Reference" "J22"
 			(at 58.42 94.234 90)
 			(effects
@@
 			(project "6502sbc"
 				(path "/dc8636f6-e59e-4c75-ae27-408ad57a23de/5a0be038-7c3c-4556-9482-35a902da59e6"
-					(reference "J21")
+					(reference "J22")
 					(unit 1)
 				)
@@
 		(dnp no)
 		(fields_autoplaced yes)
-		(property "Reference" "J22"
+		(property "Reference" "J23"
 			(at 147.32 48.26 0)
 			(effects
@@
 			(project ""
 				(path "/dc8636f6-e59e-4c75-ae27-408ad57a23de/5a0be038-7c3c-4556-9482-35a902da59e6"
-					(reference "J22")
+					(reference "J23")
 					(unit 1)
 				)
@@
 		(dnp no)
 		(fields_autoplaced yes)
-		(property "Reference" "#PWR0107"
+		(property "Reference" "#PWR098"
 			(at 68.58 149.86 0)
 			(effects
@@
 			(project "6502sbc"
 				(path "/dc8636f6-e59e-4c75-ae27-408ad57a23de/5a0be038-7c3c-4556-9482-35a902da59e6"
-					(reference "#PWR0107")
+					(reference "#PWR098")
 					(unit 1)
 				)
@@
 		(on_board yes)
 		(dnp no)
-		(property "Reference" "JP15"
+		(property "Reference" "JP21"
 			(at 62.23 144.526 0)
 			(effects
@@
 			(project ""
 				(path "/dc8636f6-e59e-4c75-ae27-408ad57a23de/5a0be038-7c3c-4556-9482-35a902da59e6"
-					(reference "JP15")
+					(reference "JP21")
 					(unit 1)
 				)
@@
 		(dnp no)
 		(fields_autoplaced yes)
-		(property "Reference" "#PWR0104"
+		(property "Reference" "#PWR0103"
 			(at 219.71 127 0)
 			(effects
@@
 			(project "6502sbc"
 				(path "/dc8636f6-e59e-4c75-ae27-408ad57a23de/5a0be038-7c3c-4556-9482-35a902da59e6"
-					(reference "#PWR0104")
+					(reference "#PWR0103")
 					(unit 1)
 				)
@@
 		(dnp no)
 		(fields_autoplaced yes)
-		(property "Reference" "U2"
+		(property "Reference" "U5"
 			(at 60.198 163.068 0)
 			(effects
@@
 				)
 				(path "/dc8636f6-e59e-4c75-ae27-408ad57a23de/5a0be038-7c3c-4556-9482-35a902da59e6"
-					(reference "U2")
+					(reference "U5")
 					(unit 1)
 				)
@@
 		(dnp no)
 		(fields_autoplaced yes)
-		(property "Reference" "J23"
+		(property "Reference" "J25"
 			(at 246.38 49.53 0)
 			(effects
@@
 			(project ""
 				(path "/dc8636f6-e59e-4c75-ae27-408ad57a23de/5a0be038-7c3c-4556-9482-35a902da59e6"
-					(reference "J23")
+					(reference "J25")
 					(unit 1)
 				)
@@
 		(dnp no)
 		(fields_autoplaced yes)
-		(property "Reference" "#PWR0106"
+		(property "Reference" "#PWR097"
 			(at 55.88 80.01 0)
 			(effects
@@
 			(project "6502sbc"
 				(path "/dc8636f6-e59e-4c75-ae27-408ad57a23de/5a0be038-7c3c-4556-9482-35a902da59e6"
-					(reference "#PWR0106")
+					(reference "#PWR097")
 					(unit 1)
 				)
@@
 		(dnp no)
 		(fields_autoplaced yes)
-		(property "Reference" "#PWR098"
+		(property "Reference" "#PWR0106"
 			(at 260.35 54.61 0)
 			(effects
@@
 			(project ""
 				(path "/dc8636f6-e59e-4c75-ae27-408ad57a23de/5a0be038-7c3c-4556-9482-35a902da59e6"
-					(reference "#PWR098")
+					(reference "#PWR0106")
 					(unit 1)
 				)
@@
 		(dnp no)
 		(fields_autoplaced yes)
-		(property "Reference" "U2"
+		(property "Reference" "U5"
 			(at 103.632 137.668 0)
 			(effects
@@
 				)
 				(path "/dc8636f6-e59e-4c75-ae27-408ad57a23de/5a0be038-7c3c-4556-9482-35a902da59e6"
-					(reference "U2")
+					(reference "U5")
 					(unit 2)
 				)
@@
 		(on_board yes)
 		(dnp no)
-		(property "Reference" "R27"
+		(property "Reference" "R28"
 			(at 115.57 138.43 90)
 			(effects
@@
 			(project "6502sbc"
 				(path "/dc8636f6-e59e-4c75-ae27-408ad57a23de/5a0be038-7c3c-4556-9482-35a902da59e6"
-					(reference "R27")
+					(reference "R28")
 					(unit 1)
 				)
@@
 		(on_board yes)
 		(dnp no)
-		(property "Reference" "TP6"
+		(property "Reference" "TP4"
 			(at 42.926 88.392 90)
 			(effects
@@
 			(project "6502sbc"
 				(path "/dc8636f6-e59e-4c75-ae27-408ad57a23de/5a0be038-7c3c-4556-9482-35a902da59e6"
-					(reference "TP6")
+					(reference "TP4")
 					(unit 1)
 				)
@@
 		(dnp no)
 		(fields_autoplaced yes)
-		(property "Reference" "#PWR099"
+		(property "Reference" "#PWR0107"
 			(at 264.16 62.23 0)
 			(effects
@@
 			(project ""
 				(path "/dc8636f6-e59e-4c75-ae27-408ad57a23de/5a0be038-7c3c-4556-9482-35a902da59e6"
-					(reference "#PWR099")
+					(reference "#PWR0107")
 					(unit 1)
 				)
@@
 		(dnp no)
 		(fields_autoplaced yes)
-		(property "Reference" "#PWR0101"
+		(property "Reference" "#PWR0100"
 			(at 132.08 53.34 0)
 			(effects
@@
 			(project "6502sbc"
 				(path "/dc8636f6-e59e-4c75-ae27-408ad57a23de/5a0be038-7c3c-4556-9482-35a902da59e6"
-					(reference "#PWR0101")
+					(reference "#PWR0100")
 					(unit 1)
 				)
@@
 		(on_board yes)
 		(dnp no)
-		(property "Reference" "TP3"
+		(property "Reference" "TP6"
 			(at 140.462 63.5 90)
 			(effects
@@
 			(project ""
 				(path "/dc8636f6-e59e-4c75-ae27-408ad57a23de/5a0be038-7c3c-4556-9482-35a902da59e6"
-					(reference "TP3")
+					(reference "TP6")
 					(unit 1)
 				)
@@
 		(dnp no)
 		(fields_autoplaced yes)
-		(property "Reference" "U36"
+		(property "Reference" "U10"
 			(at 59.69 49.53 0)
 			(effects
@@
 			(project "6502sbc"
 				(path "/dc8636f6-e59e-4c75-ae27-408ad57a23de/5a0be038-7c3c-4556-9482-35a902da59e6"
-					(reference "U36")
-					(unit 1)
-				)
+					(reference "U10")
+					(unit 1)
+				)

Commit message: Schematic is nearly done
Parts:
- added C89, C91: 0.1u, symbol Device:C_Polarized
- added C90, C92: 1u, symbol Device:C_Polarized
- U10, U8: footprint (none) -> Package_SO:TSSOP-8_3x3mm_P0.65mm; t_pd (ns) (none) -> 6.9
- U5: footprint (none) -> Package_SO:SOIC-14_3.9x8.7mm_P1.27mm; t_pd (ns) (none) -> 30
Connections:
- net +3V3: now also C91.1, C92.1
- net +5V: now also C89.1, C90.1
- net GND: now also C89.2, C90.2, C91.2, C92.2

Commit message: Most footprints assigned
Parts:
- C601: renamed from C89; footprint (none) -> Capacitor_SMD:C_0402_1005Metric
- C602: renamed from C91; footprint (none) -> Capacitor_SMD:C_0402_1005Metric
- C603: renamed from C90; footprint (none) -> Capacitor_SMD:C_0402_1005Metric
- C604: renamed from C92; footprint (none) -> Capacitor_SMD:C_0402_1005Metric
- D601: renamed from D2; footprint (none) -> LED_SMD:LED_0402_1005Metric
- JP601: renamed from JP21; footprint (none) -> Jumper:SolderJumper-3_P1.3mm_Bridged12_Pad1.0x1.5mm
- JP602: renamed from JP22; footprint (none) -> Jumper:SolderJumper-3_P1.3mm_Bridged12_Pad1.0x1.5mm
- R601: renamed from R28; footprint (none) -> Resistor_SMD:R_0402_1005Metric
- TP601: renamed from TP4; footprint (none) -> TestPoint:TestPoint_Pad_D1.5mm
- TP602: renamed from TP5; footprint (none) -> TestPoint:TestPoint_Pad_D1.5mm
- TP603: renamed from TP6; footprint (none) -> TestPoint:TestPoint_Pad_D1.5mm
- TP604: renamed from TP7; footprint (none) -> TestPoint:TestPoint_Pad_D1.5mm
- renumbered J22 to J601, J23 to J602, J24 to J603, J25 to J604, U5 to U106, U10 to U508, U8 to U509
Connections:
- net RESB: now reaches J601.8 (Pin_8)
- net DMA Peripheral Interface Module/~{RESB}: now reaches J602.8 (Pin_8)
- no-connect marks 2 -> 0
Other:
- sheet DMA Peripheral Interface Module ports: added 6502_A0, 6502_A1, 6502_A10, 6502_A2, 6502_A3, 6502_A4, 6502_A5, 6502_A6, 6502_A7, 6502_A8, 6502_A9, 6502_D0, 6502_D1, 6502_D2, 6502_D3, 6502_D4, 6502_D5, 6502_D6, 6502_D7, 6502_RW, ~{RESB}; removed 6502_{RW A0 A1 A2 A3 A4 A5 A6 A7 A8 A9 A10 D0 D1 D2 D3 D4 D5 D6 D7}
