File: hardware/6502sbc/addr_decode.kicad_sch (KiCad schematic)
At the start: 8 parts, among them U1 74AHC2G00, U14 74AHC2G00, U15 74AHC08D-Q100J, U16 CD74HC4002M96, U17 CD74HC4002M96, U18 74AHC08D-Q100J, U19 74AHC2G00, U24 CD74HC4002M96

Commit message: Preliminary schematic
Parts:
- renumbered U19 to U23, U14 to U24, U1 to U25, U15 to U26, U16 to U27, U17 to U28, U18 to U29, U24 to U9
Changed lines of the file:
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@@
 		(dnp no)
 		(fields_autoplaced yes)
-		(property "Reference" "U18"
+		(property "Reference" "U29"
 			(at 156.21 176.5299 0)
 			(effects
@@
 			(project "6502sbc"
 				(path "/dc8636f6-e59e-4c75-ae27-408ad57a23de/e68108d2-bd45-499f-89a8-24bd07fc791b"
-					(reference "U18")
+					(reference "U29")
 					(unit 5)
 				)
@@
 		(on_board yes)
 		(dnp no)
-		(property "Reference" "U14"
+		(property "Reference" "U24"
 			(at 79.248 126.492 0)
 			(effects
@@
 			(project ""
 				(path "/dc8636f6-e59e-4c75-ae27-408ad57a23de/e68108d2-bd45-499f-89a8-24bd07fc791b"
-					(reference "U14")
+					(reference "U24")
 					(unit 2)
 				)
@@
 		(on_board yes)
 		(dnp no)
-		(property "Reference" "U15"
+		(property "Reference" "U26"
 			(at 200.406 94.742 0)
 			(effects
@@
 			(project "6502sbc"
 				(path "/dc8636f6-e59e-4c75-ae27-408ad57a23de/e68108d2-bd45-499f-89a8-24bd07fc791b"
-					(reference "U15")
+					(reference "U26")
 					(unit 2)
 				)
@@
 		(on_board yes)
 		(dnp no)
-		(property "Reference" "U15"
+		(property "Reference" "U26"
 			(at 182.118 81.28 0)
 			(effects
@@
 			(project "6502sbc"
 				(path "/dc8636f6-e59e-4c75-ae27-408ad57a23de/e68108d2-bd45-499f-89a8-24bd07fc791b"
-					(reference "U15")
+					(reference "U26")
 					(unit 3)
 				)
@@
 		(dnp no)
 		(fields_autoplaced yes)
-		(property "Reference" "U19"
+		(property "Reference" "U23"
 			(at 147.3089 92.71 0)
 			(effects
@@
 			(project ""
 				(path "/dc8636f6-e59e-4c75-ae27-408ad57a23de/e68108d2-bd45-499f-89a8-24bd07fc791b"
-					(reference "U19")
+					(reference "U23")
 					(unit 1)
 				)
@@
 		(on_board yes)
 		(dnp no)
-		(property "Reference" "U1"
+		(property "Reference" "U25"
 			(at 81.534 56.388 0)
 			(effects
@@
 			(project "6502sbc"
 				(path "/dc8636f6-e59e-4c75-ae27-408ad57a23de/e68108d2-bd45-499f-89a8-24bd07fc791b"
-					(reference "U1")
+					(reference "U25")
 					(unit 2)
 				)
@@
 		(dnp no)
 		(fields_autoplaced yes)
-		(property "Reference" "U14"
+		(property "Reference" "U24"
 			(at 79.9989 96.52 0)
 			(effects
@@
 			(project ""
 				(path "/dc8636f6-e59e-4c75-ae27-408ad57a23de/e68108d2-bd45-499f-89a8-24bd07fc791b"
-					(reference "U14")
+					(reference "U24")
 					(unit 1)
 				)
@@
 		(dnp no)
 		(fields_autoplaced yes)
-		(property "Reference" "U14"
+		(property "Reference" "U24"
 			(at 31.75 175.2599 0)
 			(effects
@@
 			(project "6502sbc"
 				(path "/dc8636f6-e59e-4c75-ae27-408ad57a23de/e68108d2-bd45-499f-89a8-24bd07fc791b"
-					(reference "U14")
+					(reference "U24")
 					(unit 3)
 				)
@@
 		(dnp no)
 		(fields_autoplaced yes)
-		(property "Reference" "#PWR088"
+		(property "Reference" "#PWR0109"
 			(at 25.4 170.18 0)
 			(effects
@@
 			(project "6502sbc"
 				(path "/dc8636f6-e59e-4c75-ae27-408ad57a23de/e68108d2-bd45-499f-89a8-24bd07fc791b"
-					(reference "#PWR088")
+					(reference "#PWR0109")
 					(unit 1)
 				)
@@
 		(on_board yes)
 		(dnp no)
-		(property "Reference" "U15"
+		(property "Reference" "U26"
 			(at 59.69 175.2599 0)
 			(effects
@@
 			(project "6502sbc"
 				(path "/dc8636f6-e59e-4c75-ae27-408ad57a23de/e68108d2-bd45-499f-89a8-24bd07fc791b"
-					(reference "U15")
+					(reference "U26")
 					(unit 5)
 				)
@@
 		(on_board yes)
 		(dnp no)
-		(property "Reference" "U17"
+		(property "Reference" "U28"
 			(at 160.528 80.772 0)
 			(effects
@@
 			(project "6502sbc"
 				(path "/dc8636f6-e59e-4c75-ae27-408ad57a23de/e68108d2-bd45-499f-89a8-24bd07fc791b"
-					(reference "U17")
+					(reference "U28")
 					(unit 1)
 				)
@@
 		(dnp no)
 		(fields_autoplaced yes)
-		(property "Reference" "U16"
+		(property "Reference" "U27"
 			(at 157.48 48.26 0)
 			(effects
@@
 			(project "6502sbc"
 				(path "/dc8636f6-e59e-4c75-ae27-408ad57a23de/e68108d2-bd45-499f-89a8-24bd07fc791b"
-					(reference "U16")
+					(reference "U27")
 					(unit 1)
 				)
@@
 		(on_board yes)
 		(dnp no)
-		(property "Reference" "U16"
+		(property "Reference" "U27"
 			(at 93.98 175.8949 0)
 			(effects
@@
 			(project "6502sbc"
 				(path "/dc8636f6-e59e-4c75-ae27-408ad57a23de/e68108d2-bd45-499f-89a8-24bd07fc791b"
-					(reference "U16")
+					(reference "U27")
 					(unit 3)
 				)
@@
 		(dnp no)
 		(fields_autoplaced yes)
-		(property "Reference" "U24"
+		(property "Reference" "U9"
 			(at 107.95 96.52 0)
 			(effects
@@
 			(project ""
 				(path "/dc8636f6-e59e-4c75-ae27-408ad57a23de/e68108d2-bd45-499f-89a8-24bd07fc791b"
-					(reference "U24")
+					(reference "U9")
 					(unit 1)
 				)
@@
 		(on_board yes)
 		(dnp no)
-		(property "Reference" "U16"
+		(property "Reference" "U27"
 			(at 161.29 67.056 0)
 			(effects
@@
 			(project "6502sbc"
 				(path "/dc8636f6-e59e-4c75-ae27-408ad57a23de/e68108d2-bd45-499f-89a8-24bd07fc791b"
-					(reference "U16")
+					(reference "U27")
 					(unit 2)
 				)
@@
 		(dnp no)
 		(fields_autoplaced yes)
-		(property "Reference" "U17"
+		(property "Reference" "U28"
 			(at 125.73 175.8949 0)
 			(effects
@@
 			(project "6502sbc"
 				(path "/dc8636f6-e59e-4c75-ae27-408ad57a23de/e68108d2-bd45-499f-89a8-24bd07fc791b"
-					(reference "U17")
+					(reference "U28")
 					(unit 3)
 				)
@@
 		(on_board yes)
 		(dnp no)
-		(property "Reference" "U15"
+		(property "Reference" "U26"
 			(at 169.164 100.838 0)
 			(effects
@@
 			(project "6502sbc"
 				(path "/dc8636f6-e59e-4c75-ae27-408ad57a23de/e68108d2-bd45-499f-89a8-24bd07fc791b"
-					(reference "U15")
+					(reference "U26")
 					(unit 4)
 				)
@@
 		(dnp no)
 		(fields_autoplaced yes)
-		(property "Reference" "U1"
+		(property "Reference" "U25"
 			(at 189.2189 52.07 0)
 			(effects
@@
 			(project "6502sbc"
 				(path "/dc8636f6-e59e-4c75-ae27-408ad57a23de/e68108d2-bd45-499f-89a8-24bd07fc791b"
-					(reference "U1")
+					(reference "U25")
 					(unit 1)
 				)
@@
 		(dnp no)
 		(fields_autoplaced yes)
-		(property "Reference" "U1"
+		(property "Reference" "U25"
 			(at 33.02 137.1599 0)
 			(effects
@@
 			(project "6502sbc"
 				(path "/dc8636f6-e59e-4c75-ae27-408ad57a23de/e68108d2-bd45-499f-89a8-24bd07fc791b"
-					(reference "U1")
+					(reference "U25")
 					(unit 3)
 				)
@@
 		(dnp no)
 		(fields_autoplaced yes)
-		(property "Reference" "U15"
+		(property "Reference" "U26"
 			(at 80.0017 73.66 0)
 			(effects
@@
 			(project "6502sbc"
 				(path "/dc8636f6-e59e-4c75-ae27-408ad57a23de/e68108d2-bd45-499f-89a8-24bd07fc791b"
-					(reference "U15")
+					(reference "U26")
 					(unit 1)
 				)
@@
 		(on_board yes)
 		(dnp no)
-		(property "Reference" "U17"
+		(property "Reference" "U28"
 			(at 159.004 122.428 90)
 			(effects
@@
 			(project "6502sbc"
 				(path "/dc8636f6-e59e-4c75-ae27-408ad57a23de/e68108d2-bd45-499f-89a8-24bd07fc791b"
-					(reference "U17")
+					(reference "U28")
 					(unit 2)
 				)
@@
 		(dnp no)
 		(fields_autoplaced yes)
-		(property "Reference" "#PWR087"
+		(property "Reference" "#PWR0110"
 			(at 25.4 193.04 0)
 			(effects
@@
 			(project "6502sbc"
 				(path "/dc8636f6-e59e-4c75-ae27-408ad57a23de/e68108d2-bd45-499f-89a8-24bd07fc791b"
-					(reference "#PWR087")
+					(reference "#PWR0110")
 					(unit 1)
 				)

Commit message: Schematic is nearly done
Parts:
- U26, U29: footprint (none) -> Package_SO:SOIC-14_3.9x8.7mm_P1.27mm; t_pd (ns) (none) -> 5.9
- U27, U28, U9: t_pd (ns) (none) -> 8
Changed lines of the file:
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@@
 			)
 		)
-		(property "Footprint" ""
+		(property "Footprint" "Package_SO:SOIC-14_3.9x8.7mm_P1.27mm"
 			(at 149.86 177.8 0)
 			(effects
@@
 			)
 		)
-		(property "Datasheet" "http://www.ti.com/lit/gpn/sn74LS08"
+		(property "Datasheet" "https://assets.nexperia.com/documents/data-sheet/74AHC_AHCT08_Q100.pdf"
 			(at 149.86 177.8 0)
 			(effects
@@
 		)
 		(property "Description" "Quad And2"
+			(at 149.86 177.8 0)
+			(effects
+				(font
+					(size 1.27 1.27)
+				)
+				(hide yes)
+			)
+		)
+		(property "t_pd (ns)" "5.9"
 			(at 149.86 177.8 0)
 			(effects
@@
 			)
 		)
+		(property "t_pd (ns)" ""
+			(at 81.28 118.11 0)
+			(effects
+				(font
+					(size 1.27 1.27)
+				)
+				(hide yes)
+			)
+		)
 		(pin "8"
 		)
@@
 			)
 		)
-		(property "Footprint" ""
+		(property "Footprint" "Package_SO:SOIC-14_3.9x8.7mm_P1.27mm"
 			(at 195.58 90.17 0)
 			(effects
@@
 			)
 		)
-		(property "Datasheet" "http://www.ti.com/lit/gpn/sn74LS08"
+		(property "Datasheet" "https://assets.nexperia.com/documents/data-sheet/74AHC_AHCT08_Q100.pdf"
 			(at 195.58 90.17 0)
 			(effects
@@
 		)
 		(property "Description" "Quad And2"
+			(at 195.58 90.17 0)
+			(effects
+				(font
+					(size 1.27 1.27)
+				)
+				(hide yes)
+			)
+		)
+		(property "t_pd (ns)" "5.9"
 			(at 195.58 90.17 0)
 			(effects
@@
 			)
 		)
-		(property "Footprint" ""
+		(property "Footprint" "Package_SO:SOIC-14_3.9x8.7mm_P1.27mm"
 			(at 176.53 87.63 0)
 			(effects
@@
 			)
 		)
-		(property "Datasheet" "http://www.ti.com/lit/gpn/sn74LS08"
+		(property "Datasheet" "https://assets.nexperia.com/documents/data-sheet/74AHC_AHCT08_Q100.pdf"
 			(at 176.53 87.63 0)
 			(effects
@@
 		)
 		(property "Description" "Quad And2"
+			(at 176.53 87.63 0)
+			(effects
+				(font
+					(size 1.27 1.27)
+				)
+				(hide yes)
+			)
+		)
+		(property "t_pd (ns)" "5.9"
 			(at 176.53 87.63 0)
 			(effects
@@
 			)
 		)
+		(property "t_pd (ns)" ""
+			(at 148.59 102.87 0)
+			(effects
+				(font
+					(size 1.27 1.27)
+				)
+				(hide yes)
+			)
+		)
 		(pin "6"
 		)
@@
 			)
 		)
+		(property "t_pd (ns)" ""
+			(at 83.82 66.04 0)
+			(effects
+				(font
+					(size 1.27 1.27)
+				)
+				(hide yes)
+			)
+		)
 		(pin "3"
 		)
@@
 			)
 		)
+		(property "t_pd (ns)" ""
+			(at 81.28 106.68 0)
+			(effects
+				(font
+					(size 1.27 1.27)
+				)
+				(hide yes)
+			)
+		)
 		(pin "8"
 		)
@@
 			)
 		)
+		(property "t_pd (ns)" ""
+			(at 25.4 176.53 0)
+			(effects
+				(font
+					(size 1.27 1.27)
+				)
+				(hide yes)
+			)
+		)
 		(pin "3"
 		)
@@
 			)
 		)
-		(property "Footprint" ""
+		(property "Footprint" "Package_SO:SOIC-14_3.9x8.7mm_P1.27mm"
 			(at 53.34 176.53 0)
 			(effects
@@
 			)
 		)
-		(property "Datasheet" "http://www.ti.com/lit/gpn/sn74LS08"
+		(property "Datasheet" "https://assets.nexperia.com/documents/data-sheet/74AHC_AHCT08_Q100.pdf"
 			(at 53.34 176.53 0)
 			(effects
@@
 		)
 		(property "Description" "Quad And2"
+			(at 53.34 176.53 0)
+			(effects
+				(font
+					(size 1.27 1.27)
+				)
+				(hide yes)
+			)
+		)
+		(property "t_pd (ns)" "5.9"
 			(at 53.34 176.53 0)
 			(effects
@@
 			)
 		)
-		(property "Datasheet" ""
+		(property "Datasheet" "https://www.ti.com/lit/ds/symlink/cd54hc4002.pdf"
 			(at 153.67 87.63 0)
 			(effects
@@
 		)
 		(property "Description" ""
+			(at 153.67 87.63 0)
+			(effects
+				(font
+					(size 1.27 1.27)
+				)
+				(hide yes)
+			)
+		)
+		(property "t_pd (ns)" "8"
 			(at 153.67 87.63 0)
 			(effects
@@
 			)
 		)
-		(property "Datasheet" ""
+		(property "Datasheet" "https://www.ti.com/lit/ds/symlink/cd54hc4002.pdf"
 			(at 153.67 59.69 0)
 			(effects
@@
 		)
 		(property "Description" ""
+			(at 153.67 59.69 0)
+			(effects
+				(font
+					(size 1.27 1.27)
+				)
+				(hide yes)
+			)
+		)
+		(property "t_pd (ns)" "8"
 			(at 153.67 59.69 0)
 			(effects
@@
 			)
 		)
-		(property "Datasheet" ""
+		(property "Datasheet" "https://www.ti.com/lit/ds/symlink/cd54hc4002.pdf"
 			(at 86.36 176.53 0)
 			(effects
@@
 		)
 		(property "Description" ""
+			(at 86.36 176.53 0)
+			(effects
+				(font
+					(size 1.27 1.27)
+				)
+				(hide yes)
+			)
+		)
+		(property "t_pd (ns)" "8"
 			(at 86.36 176.53 0)
 			(effects
@@
 			)
 		)
-		(property "Datasheet" ""
+		(property "Datasheet" "https://www.ti.com/lit/ds/symlink/cd54hc4002.pdf"
 			(at 104.14 107.95 0)
 			(effects
@@
 		)
 		(property "Description" ""
+			(at 104.14 107.95 0)
+			(effects
+				(font
+					(size 1.27 1.27)
+				)
+				(hide yes)
+			)
+		)
+		(property "t_pd (ns)" "8"
 			(at 104.14 107.95 0)
 			(effects
@@
 			)
 		)
-		(property "Datasheet" ""
+		(property "Datasheet" "https://www.ti.com/lit/ds/symlink/cd54hc4002.pdf"
 			(at 156.21 73.66 0)
 			(effects
@@
 		)
 		(property "Description" ""
+			(at 156.21 73.66 0)
+			(effects
+				(font
+					(size 1.27 1.27)
+				)
+				(hide yes)
+			)
+		)
+		(property "t_pd (ns)" "8"
 			(at 156.21 73.66 0)
 			(effects
@@
 			)
 		)
-		(property "Datasheet" ""
+		(property "Datasheet" "https://www.ti.com/lit/ds/symlink/cd54hc4002.pdf"
 			(at 118.11 176.53 0)
 			(effects
@@
 		)
 		(property "Description" ""
+			(at 118.11 176.53 0)
+			(effects
+				(font
+					(size 1.27 1.27)
+				)
+				(hide yes)
+			)
+		)
+		(property "t_pd (ns)" "8"
 			(at 118.11 176.53 0)
 			(effects
@@
 			)
 		)
-		(property "Footprint" ""
+		(property "Footprint" "Package_SO:SOIC-14_3.9x8.7mm_P1.27mm"
 			(at 173.99 102.87 0)
 			(effects
@@
 			)
 		)
-		(property "Datasheet" "http://www.ti.com/lit/gpn/sn74LS08"
+		(property "Datasheet" "https://assets.nexperia.com/documents/data-sheet/74AHC_AHCT08_Q100.pdf"
 			(at 173.99 102.87 0)
 			(effects
@@
 		)
 		(property "Description" "Quad And2"
+			(at 173.99 102.87 0)
+			(effects
+				(font
+					(size 1.27 1.27)
+				)
+				(hide yes)
+			)
+		)
+		(property "t_pd (ns)" "5.9"
 			(at 173.99 102.87 0)
 			(effects
@@
 			)
 		)
+		(property "t_pd (ns)" ""
+			(at 190.5 62.23 0)
+			(effects
+				(font
+					(size 1.27 1.27)
+				)
+				(hide yes)
+			)
+		)
 		(pin "3"
 		)
@@
 			)
 		)
+		(property "t_pd (ns)" ""
+			(at 26.67 138.43 0)
+			(effects
+				(font
+					(size 1.27 1.27)
+				)
+				(hide yes)
+			)
+		)
 		(pin "8"
 		)
@@
 			)
 		)
-		(property "Footprint" ""
+		(property "Footprint" "Package_SO:SOIC-14_3.9x8.7mm_P1.27mm"
 			(at 80.01 82.55 0)
 			(effects
@@
 			)
 		)
-		(property "Datasheet" "http://www.ti.com/lit/gpn/sn74LS08"
+		(property "Datasheet" "https://assets.nexperia.com/documents/data-sheet/74AHC_AHCT08_Q100.pdf"
 			(at 80.01 82.55 0)
 			(effects
@@
 		)
 		(property "Description" "Quad And2"
+			(at 80.01 82.55 0)
+			(effects
+				(font
+					(size 1.27 1.27)
+				)
+				(hide yes)
+			)
+		)
+		(property "t_pd (ns)" "5.9"
 			(at 80.01 82.55 0)
 			(effects
@@
 			)
 		)
-		(property "Datasheet" ""
+		(property "Datasheet" "https://www.ti.com/lit/ds/symlink/cd54hc4002.pdf"
 			(at 166.37 120.65 0)
 			(effects
@@
 			(effects
 				(font
+					(size 1.27 1.27)
+				)
+				(hide yes)
+			)
+		)
+		(property "t_pd (ns)" "8"
+			(at 166.37 120.65 90)
+			(effects
+				(font

Commit message: Most footprints assigned
Parts:
- added C701, C702, C703, C704, C705, C706: .1u, Capacitor_SMD:C_0402_1005Metric, symbol Device:C
- U503: renamed from U23; footprint (none) -> Package_SO:TSSOP-8_3x3mm_P0.65mm
- U701: renamed from U24; footprint (none) -> Package_SO:TSSOP-8_3x3mm_P0.65mm
- U702: renamed from U25; footprint (none) -> Package_SO:TSSOP-8_3x3mm_P0.65mm
- renumbered U9 to U507, U26 to U703, U27 to U704, U28 to U705, U29 to U706
Connections:
- net +5V: now also U702.8 (VCC), U703.14 (VCC), U704.14 (VCC), U705.14 (VCC), U706.14 (VCC), C701.1, C702.1, C703.1, C704.1, C705.1, C706.1
- net GND: now also U702.4 (GND), U703.7 (GND), U704.7 (GND), U705.7 (GND), U706.7 (GND), C701.2, C702.2, C703.2, C704.2, C705.2, C706.2
Other:
- moved on the sheet: U702C, U704C
