File: hardware/6502sbc/bank_sel.kicad_sch (KiCad schematic)
At the start: 26 parts, among them J25 ADDRMSB_5vTTL, J26 ADDRMSB_5vCMOS, U29 74ACT139, U30 SN74ABT574ADWR, U31 SN74ABT574ADWR, U32 SN74ABT574ADWR, U33 SN74ABT574ADWR, U34 MM74HCT541MTCX

Commit message: Preliminary schematic
Parts:
- added C60, C62: .01u, symbol Device:C
- added U48: SN74ABT574ADWR, symbol 74xx:74HCT574
- added U49: 74HC04, symbol 74xx:74HC04
- renumbered C37 to C30, C30 to C31, C31 to C32, C32 to C33, C33 to C34, C34 to C35, C35 to C36, C36 to C37, J25 to J26, J26 to J27, JP21 to JP23, R30 to R29, R31 to R30, R32 to R31, R33 to R32, R34 to R33, R35 to R34, R36 to R35, R37 to R36, R38 to R37, U29 to U30, U30 to U31, U31 to U32, U32 to U33, U33 to U34, U34 to U35
Connections:
- net +5V: now also C60.2, C62.1, U48.20 (VCC), U49.14 (VCC)
- net D0: now also U48.2 (D0)
- net D1: now also U48.3 (D1)
- net D2: now also U48.4 (D2)
- net D3: now also U48.5 (D3)
- net D4: now also U48.6 (D4)
- net D5: now also U48.7 (D5)
- net D6: now also U48.8 (D6)
- net D7: now also U48.9 (D7)
- net GND: now also C60.1, C62.2, U48.1 (OE), U48.10 (GND), U49.11, U49.13, U49.7 (GND)
- net at U34.11 (Cp): now also U49.6; no longer U30.10 (O2)
- net at U30.11 (O1): now also U49.3; no longer U33.11 (Cp)
- net at U30.12 (O0): now also U49.1; no longer U32.11 (Cp)
- net at U30.9 (O3): now also U49.9; no longer U31.11 (Cp)
- new net: U30.10 (O2), U49.5
- new net: U32.11 (Cp), U49.2
- new net: U33.11 (Cp), U49.4
- new net: U31.11 (Cp), U49.8
- new net B20: U48.19 (Q0)
- new net B21: U48.18 (Q1)
- new net B22: U48.17 (Q2)
- new net B23: U48.16 (Q3)
- new net B24: U48.15 (Q4)
- new net B25: U48.14 (Q5)
- new net B26: U48.13 (Q6)
- new net B27: U48.12 (Q7)
- new net WBANKCK2: U48.11 (Cp)
- no-connect marks 0 -> 2
Other:
- note added: "Pull-downs to avoid Hi-Z — thus, high-mem is always bank 0"
- note added: "Should I just get the right clock deocder instead of using a bunch of inverters?"
- note removed: "Pull-downs to avoid Hi-Z in case of deocder malfunction And to reduce hazards in transitions"
- moved on the sheet: U30B

Commit message: Schematic is nearly done
Parts:
- removed unit 6 of U49
- U49: footprint (none) -> Package_SO:SOIC-14_3.9x8.7mm_P1.27mm; t_pd (ns) (none) -> 19
Connections:
- no-connect marks 2 -> 1
Other:
- note removed: "Should I just get the right clock deocder instead of using a bunch of inverters?"

Commit message: Most footprints assigned
Parts:
- C801: renamed from C30; footprint (none) -> Capacitor_SMD:C_0402_1005Metric
- C802: renamed from C31; footprint (none) -> Capacitor_SMD:C_0402_1005Metric
- C803: renamed from C62; footprint (none) -> Capacitor_SMD:C_0402_1005Metric
- C804: renamed from C32; footprint (none) -> Capacitor_SMD:C_0402_1005Metric
- C805: renamed from C33; footprint (none) -> Capacitor_SMD:C_0402_1005Metric
- C806: renamed from C34; footprint (none) -> Capacitor_SMD:C_0402_1005Metric
- C807: renamed from C35; footprint (none) -> Capacitor_SMD:C_0402_1005Metric
- C808: renamed from C60; footprint (none) -> Capacitor_SMD:C_0402_1005Metric
- JP801: renamed from JP23; footprint (none) -> Jumper:SolderJumper-2_P1.3mm_Open_Pad1.0x1.5mm
- R801: renamed from R29; footprint (none) -> Resistor_SMD:R_0402_1005Metric
- R802: renamed from R30; footprint (none) -> Resistor_SMD:R_0402_1005Metric
- R803: renamed from R31; footprint (none) -> Resistor_SMD:R_0402_1005Metric
- R804: renamed from R32; footprint (none) -> Resistor_SMD:R_0402_1005Metric
- R805: renamed from R33; footprint (none) -> Resistor_SMD:R_0402_1005Metric
- R806: renamed from R34; footprint (none) -> Resistor_SMD:R_0402_1005Metric
- R807: renamed from R35; footprint (none) -> Resistor_SMD:R_0402_1005Metric
- R808: renamed from R36; footprint (none) -> Resistor_SMD:R_0402_1005Metric
- R809: renamed from R37; footprint (none) -> Resistor_SMD:R_0402_1005Metric
- U801: renamed from U30; footprint (none) -> Package_SO:TSSOP-16_4.4x5mm_P0.65mm
- U802: renamed from U31; value SN74ABT574ADWR -> SN74ABT574APWR; footprint (none) -> Package_SO:TSSOP-20_4.4x6.5mm_P0.65mm
- U803: renamed from U32; value SN74ABT574ADWR -> SN74ABT574APWR; footprint (none) -> Package_SO:TSSOP-20_4.4x6.5mm_P0.65mm
- U804: renamed from U33; value SN74ABT574ADWR -> SN74ABT574APWR; footprint (none) -> Package_SO:TSSOP-20_4.4x6.5mm_P0.65mm
- U805: renamed from U34; value SN74ABT574ADWR -> SN74ABT574APWR; footprint (none) -> Package_SO:TSSOP-20_4.4x6.5mm_P0.65mm
- U806: renamed from U48; value SN74ABT574ADWR -> SN74ABT574APWR; footprint (none) -> Package_SO:TSSOP-20_4.4x6.5mm_P0.65mm
- renumbered C36 to C809, C37 to C810, J26 to J801, J27 to J802, U49 to U109, U35 to U807
