File: hardware/6502sbc/dma_pi.kicad_sch (KiCad schematic)
At the start: 47 parts, among them J1 ICSP Header, J10 UART, J11 SPI BUS, J2 EXT INT, J3 PeripheralBusB, J4 PeripheralBusA, J5 PIC_PORTD, J6 SmartPeripheral, J7 SmartPeripheral, J8 SPI AUX, J9 I2C BUS, U7 SN74LS07, U9 PIC16F15385-xPT, Y1 NOPOP

Commit message: Preliminary schematic
Parts:
- renumbered C11 to C10, C16 to C11, C17 to C12, C18 to C13, C19 to C14, C8 to C7, C9 to C8, C10 to C9, J8 to J10, J9 to J11, J10 to J12, J11 to J13, J1 to J3, J2 to J4, J3 to J5, J4 to J6, J5 to J7, J6 to J8, J7 to J9, JP6 to JP10, JP7 to JP11, JP8 to JP12, JP9 to JP13, JP10 to JP14, JP11 to JP15, JP1 to JP7, JP2 to JP8, JP5 to JP9, R5 to R10, R6 to R11, R7 to R12, R8 to R13, R9 to R14, R10 to R15, R11 to R16, R12 to R17, R13 to R18, R2 to R7, R3 to R8, R4 to R9, TP2 to TP3, U7 to U12, U8 to U13, U9 to U14

Commit message: Schematic is nearly done
Parts:
- removed J6: PeripheralBusA, symbol Connector:Conn_01x08_Pin
- removed J8, J9: SmartPeripheral, symbol Connector_Generic:Conn_02x04_Counter_Clockwise
- added C83, C84: 1u, symbol Device:C
- added C85, C88: 1u, symbol Device:C_Polarized
- added C86, C87: 0.1u, symbol Device:C_Polarized
- added J14: Conn_01x02_Pin, symbol Connector:Conn_01x02_Pin
- added J6: I2C, symbol Connector:Conn_01x05_Pin
- added J8, J9: Conn_02x05_Counter_Clockwise, symbol Connector_Generic:Conn_02x05_Counter_Clockwise
- added R79, R80, R81, R82, R83, R84, R85, R86: 33, symbol Device:R
- C10, C13: value .01u -> .1u
- C11, C14: value .1u -> .01u
- C12: value 10n -> .01u
- U12: t_pd (ns) (none) -> 30
- U13: value ~ -> CY7C146-25JC
Connections:
- net KEY_INT is gone; now on net AUX_INT1: J5.3 (Pin_3), U12.3
- net +3V3: now also J6.1 (Pin_1), J8.8 (Pin_8), J9.8 (Pin_8)
- net +5V: now also C83.1, C84.1, C85.1, C86.1, C87.1, C88.1, J6.2 (Pin_2), J8.9 (Pin_9), J9.9 (Pin_9)
- net 6502_D0: now also R79.1; no longer U13.17 (D0_L)
- net 6502_D1: now also R80.1; no longer U13.18 (D1_L)
- net 6502_D2: now also R81.1; no longer U13.19 (D2_L)
- net 6502_D3: now also R82.1; no longer U13.20 (D3_L)
- net 6502_D4: now also R83.1; no longer U13.21 (D4_L)
- net 6502_D5: now also R84.1; no longer U13.22 (D5_L)
- net 6502_D6: now also R85.1; no longer U13.23 (D6_L)
- net 6502_D7: now also R86.1; no longer U13.24 (D7_L)
- net GND: now also J5.5 (Pin_5), C83.2, C84.2, C85.2, C86.2, C87.2, C88.2, J14.1 (Pin_1), J6.5 (Pin_5), J8.10 (Pin_10), J8.3 (Pin_3), J8.6 (Pin_6), J8.7 (Pin_7), J9.10 (Pin_10), J9.3 (Pin_3), J9.6 (Pin_6), J9.7 (Pin_7)
- net SCL: now also J6.4 (Pin_4), J8.2 (Pin_2), J9.2 (Pin_2)
- net SDA: now also J6.3 (Pin_3), J8.1 (Pin_1), J9.1 (Pin_1)
- net SS_AUX: now also J5.4 (Pin_4); no longer J5.5 (Pin_5)
- net SS_MEM: no longer J5.4 (Pin_4)
- net UARTrx: now also J8.5 (Pin_5), J9.5 (Pin_5)
- net UARTtx: now also J8.4 (Pin_4), J9.4 (Pin_4)
- net PIC Peripherals/OC_MOSI: now reaches U12.10
- net PIC Peripherals/OC_SS_SD: now reaches U12.8
- net PIC Peripherals/OC_SCK: now reaches U12.12
- net AUX_INT renamed AUX_INT1
- net AUX_INT1: no longer U12.5
- new net: R79.2, U13.17 (D0_L)
- new net: R80.2, U13.18 (D1_L)
- new net: R81.2, U13.19 (D2_L)
- new net: R82.2, U13.20 (D3_L)
- new net: R83.2, U13.21 (D4_L)
- new net: R84.2, U13.22 (D5_L)
- new net: R85.2, U13.23 (D6_L)
- new net: R86.2, U13.24 (D7_L)
- new net AUX_INT2: J14.2 (Pin_2), U12.5
Other:
- sheet PIC Peripherals ports: added OC_MOSI, OC_SCK, OC_SS_SD, P_MISO, P_MOSI, P_SCK, P_SS_MEM; removed none
- note added: "Peripherals"
- note removed: "(Separate Submodule)"
- note removed: "Peripheral Interface"
- note removed: "Tank Capacitor"
- moved on the sheet: C5, J3, J4, J5, R11, R12, U12D, U12E, U12F

Commit message: Most footprints assigned
Parts:
- removed J14: Conn_01x02_Pin, symbol Connector:Conn_01x02_Pin
- removed J7: PIC_PORTD, symbol Connector:Conn_01x08_Pin
- added J205: Conn_01x09_Pin, symbol Connector:Conn_01x09_Pin
- added R221: 4.7k, Resistor_SMD:R_0402_1005Metric, symbol Device:R
- C201: renamed from C5; footprint (none) -> Capacitor_SMD:C_0402_1005Metric
- C202: renamed from C6; footprint (none) -> Capacitor_SMD:C_0402_1005Metric
- C203: renamed from C7; footprint (none) -> Capacitor_SMD:C_0402_1005Metric
- C204: renamed from C8; footprint (none) -> Capacitor_SMD:C_0402_1005Metric
- C205: renamed from C9; footprint (none) -> Capacitor_SMD:C_0402_1005Metric
- C206: renamed from C87; footprint (none) -> Capacitor_SMD:C_0402_1005Metric
- C207: renamed from C83; footprint (none) -> Capacitor_SMD:C_0402_1005Metric
- C208: renamed from C10; footprint (none) -> Capacitor_SMD:C_0402_1005Metric
- C209: renamed from C11; footprint (none) -> Capacitor_SMD:C_0402_1005Metric
- C210: renamed from C88; footprint (none) -> Capacitor_SMD:C_0402_1005Metric
- C211: renamed from C86; footprint (none) -> Capacitor_SMD:C_0402_1005Metric
- C212: renamed from C85; footprint (none) -> Capacitor_SMD:C_0402_1005Metric
- C213: renamed from C12; footprint (none) -> Capacitor_SMD:C_0402_1005Metric
- C214: renamed from C84; footprint (none) -> Capacitor_SMD:C_0402_1005Metric
- C215: renamed from C13; footprint (none) -> Capacitor_SMD:C_0402_1005Metric
- C216: renamed from C14; footprint (none) -> Capacitor_SMD:C_0402_1005Metric
- JP201: renamed from JP7; footprint (none) -> Jumper:SolderJumper-2_P1.3mm_Bridged2Bar_Pad1.0x1.5mm
- JP202: renamed from JP8; footprint (none) -> Jumper:SolderJumper-2_P1.3mm_Open_Pad1.0x1.5mm
- JP203: renamed from JP9; footprint (none) -> Jumper:SolderJumper-2_P1.3mm_Bridged2Bar_Pad1.0x1.5mm
- JP204: renamed from JP10; footprint (none) -> Jumper:SolderJumper-2_P1.3mm_Open_Pad1.0x1.5mm
- JP205: renamed from JP11; footprint (none) -> Jumper:SolderJumper-2_P1.3mm_Bridged2Bar_Pad1.0x1.5mm
- JP206: renamed from JP12; footprint (none) -> Jumper:SolderJumper-2_P1.3mm_Bridged2Bar_Pad1.0x1.5mm
- JP207: renamed from JP13; footprint (none) -> Jumper:SolderJumper-2_P1.3mm_Bridged2Bar_Pad1.0x1.5mm
- JP208: renamed from JP14; footprint (none) -> Jumper:SolderJumper-2_P1.3mm_Open_Pad1.0x1.5mm
- JP209: renamed from JP15; footprint (none) -> Jumper:SolderJumper-3_P1.3mm_Bridged12_Pad1.0x1.5mm
- R201: renamed from R7; footprint (none) -> Resistor_SMD:R_0402_1005Metric
- R202: renamed from R8; footprint (none) -> Resistor_SMD:R_0402_1005Metric
- R203: renamed from R9; footprint (none) -> Resistor_SMD:R_0402_1005Metric
- R204: renamed from R10; footprint (none) -> Resistor_SMD:R_0402_1005Metric
- R205: renamed from R79; footprint (none) -> Resistor_SMD:R_0402_1005Metric
- R206: renamed from R80; footprint (none) -> Resistor_SMD:R_0402_1005Metric
- R207: renamed from R81; footprint (none) -> Resistor_SMD:R_0402_1005Metric
- R208: renamed from R82; footprint (none) -> Resistor_SMD:R_0402_1005Metric
- R209: renamed from R83; footprint (none) -> Resistor_SMD:R_0402_1005Metric
- R210: renamed from R84; footprint (none) -> Resistor_SMD:R_0402_1005Metric
- R211: renamed from R85; footprint (none) -> Resistor_SMD:R_0402_1005Metric
- R212: renamed from R86; footprint (none) -> Resistor_SMD:R_0402_1005Metric
- R213: renamed from R11; footprint (none) -> Resistor_SMD:R_0402_1005Metric
- R214: renamed from R12; footprint (none) -> Resistor_SMD:R_0402_1005Metric
- R215: renamed from R13; footprint (none) -> Resistor_SMD:R_0402_1005Metric
- R216: renamed from R14; footprint (none) -> Resistor_SMD:R_0402_1005Metric
- R217: renamed from R15; footprint (none) -> Resistor_SMD:R_0402_1005Metric
- R218: renamed from R16; footprint (none) -> Resistor_SMD:R_0402_1005Metric
- R219: renamed from R17; footprint (none) -> Resistor_SMD:R_0402_1005Metric
- R220: renamed from R18; footprint (none) -> Resistor_SMD:R_0402_1005Metric
- TP201: renamed from TP3; footprint (none) -> TestPoint:TestPoint_Pad_D1.5mm
- renumbered J3 to J201, J5 to J202, J4 to J203, J6 to J204, J8 to J206, J9 to J207, J10 to J208, J11 to J209, J12 to J210, J13 to J211, U12 to U201, U13 to U202, U14 to U203, Y1 to Y201
Connections:
- net AUX_SEL: now also JP204.2 (B), U203.2 (RD4), J205.6 (Pin_6); no longer U203.22 (RA1)
- net GND: now also J205.1 (Pin_1), R221.2
- net PIC_INT: no longer U201.6
- net at JP205.2 (B), JP208.1 (A), U203.3 (RD5): now also J205.7 (Pin_7)
- net at JP207.1 (A), U203.4 (RD6): now also J205.8 (Pin_8)
- net at U203.42 (RD0): now also J205.2 (Pin_2)
- net at U203.43 (RD1): now also J205.3 (Pin_3)
- net at U203.44 (RD2): now also J205.4 (Pin_4)
- net at U203.45 (RD3): now also J205.5 (Pin_5)
- net at JP206.1 (A), U203.5 (RD7): now also J205.9 (Pin_9)
- net AUX_INT2: no longer names the net of U201.5
- net AUX_INT2: now also U203.22 (RA1), R221.1
- new net ~{RESB}: U201.6
Other:
- note added: "To reset the CPU"
- note removed: "6502 BUS"
- note removed: "Ext Input"
- moved on the sheet: U201C
