File: hardware/6502sbc/peripherals.kicad_sch (KiCad schematic)
At the start: 34 parts, among them J12 PeripheralBusA, J13 SD CARD, J14 AUX SS, J15 PeripheralBusB, J18 Micro_SD_Card, J19 KMDGX-6S-BS, U10 74HCT125D, U11 74HC04, U12 M95512-Axxx-MF, U13 74HC595, U22 74HC193, U23 PCF8574T

Commit message: Preliminary schematic
Parts:
- renumbered C20 to C15, C21 to C16, C22 to C17, C23 to C18, C24 to C19, C25 to C20, C26 to C21, C27 to C22, C28 to C23, C29 to C24, J12 to J14, J13 to J15, J14 to J16, J15 to J17, JP12 to JP16, JP13 to JP17, JP14 to JP18, R14 to R19, R15 to R20, R16 to R21, R17 to R22, R18 to R23, U10 to U15, U12 to U16, U11 to U17, U13 to U18, U22 to U19, U23 to U20

Commit message: Schematic is nearly done
Parts:
- removed J14: PeripheralBusA, symbol Connector:Conn_01x08_Pin
- removed J16: AUX SS, symbol Connector:Conn_01x02_Pin
- removed J17: PeripheralBusB, symbol Connector:Conn_01x08_Pin
- C15, C17: value .01u -> 1u
- U17: footprint (none) -> Package_SO:SOIC-14_3.9x8.7mm_P1.27mm; t_pd (ns) (none) -> 19
Other:
- note added: "(Excluded from board; It is better to have the PS/2 interface by the CPU. No point in having extra things interrupted for each character typed.)"
- note added: "Interface from DMA Schematic"
- note removed: "Aux Slave Select"
- note removed: "Decoupling Caps"
- note removed: "I2C"
- note removed: "Interface from DMA Submodule"
- note removed: "Keyboard Interrupt (TTL or CMOS)"
- moved on the sheet: J15

Commit message: Most footprints assigned
Parts:
- removed C20: .1u, symbol Device:C
- removed C21, C22, C23, C24: .01u, symbol Device:C
- removed J19: KMDGX-6S-BS, symbol Connector:Mini-DIN-6
- removed JP16, JP17: SolderJumper_3_Bridged12, symbol Jumper:SolderJumper_3_Bridged12
- removed JP18: ADDR SEL, symbol Jumper:SolderJumper_3_Bridged12
- removed R24, R25, R26: 10k, symbol Device:R
- removed U17: 74HC04, Package_SO:SOIC-14_3.9x8.7mm_P1.27mm, symbol 74xx:74HC04
- removed U18: 74HC595, symbol 74xx:74HC595
- removed U19: 74HC193, symbol 74xx:74HC193
- removed U20: PCF8574T, Package_SO:SOIC-16W_7.5x10.3mm_P1.27mm, symbol Interface_Expansion:PCF8574T
- C401: renamed from C15; footprint (none) -> Capacitor_SMD:C_0402_1005Metric
- C402: renamed from C16; footprint (none) -> Capacitor_SMD:C_0402_1005Metric
- C403: renamed from C17; footprint (none) -> Capacitor_SMD:C_0402_1005Metric
- C404: renamed from C18; footprint (none) -> Capacitor_SMD:C_0402_1005Metric
- C405: renamed from C19; footprint (none) -> Capacitor_SMD:C_0402_1005Metric
- D401: renamed from D1; footprint (none) -> LED_SMD:LED_0402_1005Metric
- R401: renamed from R19; footprint (none) -> Resistor_SMD:R_0402_1005Metric
- R402: renamed from R20; footprint (none) -> Resistor_SMD:R_0402_1005Metric
- R403: renamed from R21; footprint (none) -> Resistor_SMD:R_0402_1005Metric
- R404: renamed from R22; footprint (none) -> Resistor_SMD:R_0402_1005Metric
- R405: renamed from R23; footprint (none) -> Resistor_SMD:R_0402_1005Metric
- renumbered J15 to J401, J18 to J402, U15 to U401, U16 to U402
Connections:
- no-connect marks 15 -> 6
Other:
- note removed: "(Excluded from board; It is better to have the PS/2 interface by the CPU. No point in having extra things interrupted for each character typed.)"
- note removed: "Clear, to accept new data"
- note removed: "I2C PS/2 Keyboard Interface"
- note removed: "add prop. delay"
