File: hardware/6502sbc/priv_except.kicad_sch (KiCad schematic)
At the start: 9 parts, among them U18 74AHC08D-Q100J, U19 74AHC2G00, U20 74AHC2G32DP, U21 74AHC08D-Q100J, U24 CD74HC4002M96, U27 74LS73

Commit message: Preliminary schematic
Parts:
- renumbered JP18 to JP24, R28 to R38, U20 to U11, U21 to U2, U19 to U23, U18 to U29, U21 to U5, U27 to U7, U24 to U9
Changed lines of the file:
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@@
 		(dnp no)
 		(fields_autoplaced yes)
-		(property "Reference" "U27"
+		(property "Reference" "U7"
 			(at 236.22 62.23 0)
 			(effects
@@
 			(project "6502sbc"
 				(path "/dc8636f6-e59e-4c75-ae27-408ad57a23de/78558388-3613-4012-b027-bd956c6e0596"
-					(reference "U27")
+					(reference "U7")
 					(unit 1)
 				)
@@
 		(dnp no)
 		(fields_autoplaced yes)
-		(property "Reference" "U21"
+		(property "Reference" "U2"
 			(at 66.0317 72.39 0)
 			(effects
@@
 			(project "6502sbc"
 				(path "/dc8636f6-e59e-4c75-ae27-408ad57a23de/78558388-3613-4012-b027-bd956c6e0596"
-					(reference "U21")
+					(reference "U2")
 					(unit 3)
 				)
@@
 		(on_board yes)
 		(dnp no)
-		(property "Reference" "U20"
+		(property "Reference" "U11"
 			(at 211.582 81.788 0)
 			(effects
@@
 			(project "6502sbc"
 				(path "/dc8636f6-e59e-4c75-ae27-408ad57a23de/78558388-3613-4012-b027-bd956c6e0596"
-					(reference "U20")
+					(reference "U11")
 					(unit 1)
 				)
@@
 		(dnp no)
 		(fields_autoplaced yes)
-		(property "Reference" "U18"
+		(property "Reference" "U29"
 			(at 43.1717 54.61 0)
 			(effects
@@
 			(project "6502sbc"
 				(path "/dc8636f6-e59e-4c75-ae27-408ad57a23de/78558388-3613-4012-b027-bd956c6e0596"
-					(reference "U18")
+					(reference "U29")
 					(unit 2)
 				)
@@
 		(dnp no)
 		(fields_autoplaced yes)
-		(property "Reference" "U18"
+		(property "Reference" "U29"
 			(at 71.1117 52.07 0)
 			(effects
@@
 			(project "6502sbc"
 				(path "/dc8636f6-e59e-4c75-ae27-408ad57a23de/78558388-3613-4012-b027-bd956c6e0596"
-					(reference "U18")
+					(reference "U29")
 					(unit 4)
 				)
@@
 		(on_board yes)
 		(dnp no)
-		(property "Reference" "R28"
+		(property "Reference" "R38"
 			(at 243.84 99.06 90)
 			(effects
@@
 			(project "6502sbc"
 				(path "/dc8636f6-e59e-4c75-ae27-408ad57a23de/78558388-3613-4012-b027-bd956c6e0596"
-					(reference "R28")
+					(reference "R38")
 					(unit 1)
 				)
@@
 		(on_board yes)
 		(dnp no)
-		(property "Reference" "U21"
+		(property "Reference" "U2"
 			(at 70.612 148.336 0)
 			(effects
@@
 			(project "6502sbc"
 				(path "/dc8636f6-e59e-4c75-ae27-408ad57a23de/78558388-3613-4012-b027-bd956c6e0596"
-					(reference "U21")
+					(reference "U2")
 					(unit 2)
 				)
@@
 		(dnp no)
 		(fields_autoplaced yes)
-		(property "Reference" "U18"
+		(property "Reference" "U29"
 			(at 43.1717 39.37 0)
 			(effects
@@
 			(project "6502sbc"
 				(path "/dc8636f6-e59e-4c75-ae27-408ad57a23de/78558388-3613-4012-b027-bd956c6e0596"
-					(reference "U18")
+					(reference "U29")
 					(unit 3)
 				)
@@
 		(on_board yes)
 		(dnp no)
-		(property "Reference" "U24"
+		(property "Reference" "U9"
 			(at 70.612 130.048 0)
 			(effects
@@
 			(project "6502sbc"
 				(path "/dc8636f6-e59e-4c75-ae27-408ad57a23de/78558388-3613-4012-b027-bd956c6e0596"
-					(reference "U24")
+					(reference "U9")
 					(unit 2)
 				)
@@
 		(dnp no)
 		(fields_autoplaced yes)
-		(property "Reference" "U20"
+		(property "Reference" "U11"
 			(at 93.98 140.97 0)
 			(effects
@@
 			(project "6502sbc"
 				(path "/dc8636f6-e59e-4c75-ae27-408ad57a23de/78558388-3613-4012-b027-bd956c6e0596"
-					(reference "U20")
+					(reference "U11")
 					(unit 2)
 				)
@@
 		(dnp no)
 		(fields_autoplaced yes)
-		(property "Reference" "U18"
+		(property "Reference" "U29"
 			(at 43.1717 69.85 0)
 			(effects
@@
 			(project "6502sbc"
 				(path "/dc8636f6-e59e-4c75-ae27-408ad57a23de/78558388-3613-4012-b027-bd956c6e0596"
-					(reference "U18")
+					(reference "U29")
 					(unit 1)
 				)
@@
 		(on_board yes)
 		(dnp no)
-		(property "Reference" "#PWR0109"
+		(property "Reference" "#PWR0135"
 			(at 238.76 95.25 0)
 			(effects
@@
 			(project "6502sbc"
 				(path "/dc8636f6-e59e-4c75-ae27-408ad57a23de/78558388-3613-4012-b027-bd956c6e0596"
-					(reference "#PWR0109")
+					(reference "#PWR0135")
 					(unit 1)
 				)
@@
 		(dnp no)
 		(fields_autoplaced yes)
-		(property "Reference" "U21"
+		(property "Reference" "U5"
 			(at 134.62 153.67 0)
 			(effects
@@
 			(project "6502sbc"
 				(path "/dc8636f6-e59e-4c75-ae27-408ad57a23de/78558388-3613-4012-b027-bd956c6e0596"
-					(reference "U21")
+					(reference "U5")
 					(unit 6)
 				)
@@
 		(dnp no)
 		(fields_autoplaced yes)
-		(property "Reference" "U27"
+		(property "Reference" "U7"
 			(at 119.38 149.86 0)
 			(effects
@@
 			(project "6502sbc"
 				(path "/dc8636f6-e59e-4c75-ae27-408ad57a23de/78558388-3613-4012-b027-bd956c6e0596"
-					(reference "U27")
+					(reference "U7")
 					(unit 2)
 				)
@@
 		(dnp no)
 		(fields_autoplaced yes)
-		(property "Reference" "#PWR0111"
+		(property "Reference" "#PWR0134"
 			(at 227.33 86.36 0)
 			(effects
@@
 			(project "6502sbc"
 				(path "/dc8636f6-e59e-4c75-ae27-408ad57a23de/78558388-3613-4012-b027-bd956c6e0596"
-					(reference "#PWR0111")
+					(reference "#PWR0134")
 					(unit 1)
 				)
@@
 		(dnp no)
 		(fields_autoplaced yes)
-		(property "Reference" "#PWR0110"
+		(property "Reference" "#PWR0133"
 			(at 120.65 167.64 0)
 			(effects
@@
 			(project "6502sbc"
 				(path "/dc8636f6-e59e-4c75-ae27-408ad57a23de/78558388-3613-4012-b027-bd956c6e0596"
-					(reference "#PWR0110")
+					(reference "#PWR0133")
 					(unit 1)
 				)
@@
 		(dnp no)
 		(fields_autoplaced yes)
-		(property "Reference" "U21"
+		(property "Reference" "U2"
 			(at 217.1617 54.61 0)
 			(effects
@@
 			(project "6502sbc"
 				(path "/dc8636f6-e59e-4c75-ae27-408ad57a23de/78558388-3613-4012-b027-bd956c6e0596"
-					(reference "U21")
+					(reference "U2")
 					(unit 1)
 				)
@@
 		(dnp no)
 		(fields_autoplaced yes)
-		(property "Reference" "U21"
+		(property "Reference" "U5"
 			(at 267.97 82.55 0)
 			(effects
@@
 			(project "6502sbc"
 				(path "/dc8636f6-e59e-4c75-ae27-408ad57a23de/78558388-3613-4012-b027-bd956c6e0596"
-					(reference "U21")
+					(reference "U5")
 					(unit 3)
 				)
@@
 		(on_board yes)
 		(dnp no)
-		(property "Reference" "JP18"
+		(property "Reference" "JP24"
 			(at 77.978 138.938 0)
 			(effects
@@
 			(project "6502sbc"
 				(path "/dc8636f6-e59e-4c75-ae27-408ad57a23de/78558388-3613-4012-b027-bd956c6e0596"
-					(reference "JP18")
+					(reference "JP24")
 					(unit 1)
 				)
@@
 		(dnp no)
 		(fields_autoplaced yes)
-		(property "Reference" "U19"
+		(property "Reference" "U23"
 			(at 87.63 96.5088 90)
 			(effects
@@
 			(project "6502sbc"
 				(path "/dc8636f6-e59e-4c75-ae27-408ad57a23de/78558388-3613-4012-b027-bd956c6e0596"
-					(reference "U19")
+					(reference "U23")
 					(unit 2)
 				)

Commit message: Schematic is nearly done
Parts:
- U11: footprint (none) -> Package_SO:TSSOP-8_3x3mm_P0.65mm; t_pd (ns) (none) -> 6.9
- U2, U29: footprint (none) -> Package_SO:SOIC-14_3.9x8.7mm_P1.27mm; t_pd (ns) (none) -> 5.9
- U5: footprint (none) -> Package_SO:SOIC-14_3.9x8.7mm_P1.27mm; t_pd (ns) (none) -> 30
- U7: value 74LS73 -> 74HC73D; footprint (none) -> Package_SO:SOIC-14_3.9x8.7mm_P1.27mm; t_pd (ns) (none) -> clk-q: 30; setup: 16; hold: 3
- U9: t_pd (ns) (none) -> 8
Connections:
- net RESPRIV: no longer U7.3 (K)
- net ~{VPB}: now also U7.3 (K)
- net FAULT: now reaches U11.3, U7.14 (J)

Commit message: Most footprints assigned
Parts:
- D901: renamed from D3; footprint (none) -> LED_SMD:LED_0402_1005Metric
- JP901: renamed from JP24; footprint (none) -> Jumper:SolderJumper-2_P1.3mm_Bridged2Bar_Pad1.0x1.5mm
- R901: renamed from R38; footprint (none) -> Resistor_SMD:R_0402_1005Metric
- U503: renamed from U23; footprint (none) -> Package_SO:TSSOP-8_3x3mm_P0.65mm
- renumbered U5 to U106, U2 to U110, U7 to U505, U9 to U507, U11 to U510, U29 to U706
Connections:
- no-connect marks 0 -> 1
Changed lines of the file:
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@@
 		)
 	)
+	(no_connect
+		(at 127 157.48)
+	)
 	(wire
 		(pts
@@
 		)
 	)
-	(label "SYNC"
-		(at 53.34 83.82 0)
-		(effects
-			(font
-				(size 1.27 1.27)
-			)
-			(justify left bottom)
-		)
-	)
 	(label "D1"
 		(at 31.75 50.8 0)
@@
 		)
 	)
+	(hierarchical_label "SYNC"
+		(shape input)
+		(at 53.34 83.82 180)
+		(effects
+			(font
+				(size 1.27 1.27)
+			)
+			(justify right)
+		)
+	)
 	(hierarchical_label "XLEVEL_KERNEL"
 		(shape output)
@@
 		(dnp no)
 		(fields_autoplaced yes)
-		(property "Reference" "U7"
+		(property "Reference" "U505"
 			(at 236.22 62.23 0)
 			(effects
@@
 			(project "6502sbc"
 				(path "/dc8636f6-e59e-4c75-ae27-408ad57a23de/78558388-3613-4012-b027-bd956c6e0596"
-					(reference "U7")
+					(reference "U505")
 					(unit 1)
 				)
@@
 		(dnp no)
 		(fields_autoplaced yes)
-		(property "Reference" "U2"
+		(property "Reference" "U110"
 			(at 66.0317 72.39 0)
 			(effects
@@
 			(project "6502sbc"
 				(path "/dc8636f6-e59e-4c75-ae27-408ad57a23de/78558388-3613-4012-b027-bd956c6e0596"
-					(reference "U2")
+					(reference "U110")
 					(unit 3)
 				)
@@
 		(on_board yes)
 		(dnp no)
-		(property "Reference" "U11"
+		(property "Reference" "U510"
 			(at 211.582 81.788 0)
 			(effects
@@
 			(project "6502sbc"
 				(path "/dc8636f6-e59e-4c75-ae27-408ad57a23de/78558388-3613-4012-b027-bd956c6e0596"
-					(reference "U11")
+					(reference "U510")
 					(unit 1)
 				)
@@
 		(dnp no)
 		(fields_autoplaced yes)
-		(property "Reference" "U29"
+		(property "Reference" "U706"
 			(at 43.1717 54.61 0)
 			(effects
@@
 			(project "6502sbc"
 				(path "/dc8636f6-e59e-4c75-ae27-408ad57a23de/78558388-3613-4012-b027-bd956c6e0596"
-					(reference "U29")
+					(reference "U706")
 					(unit 2)
 				)
@@
 		(dnp no)
 		(fields_autoplaced yes)
-		(property "Reference" "U29"
+		(property "Reference" "U706"
 			(at 71.1117 52.07 0)
 			(effects
@@
 			(project "6502sbc"
 				(path "/dc8636f6-e59e-4c75-ae27-408ad57a23de/78558388-3613-4012-b027-bd956c6e0596"
-					(reference "U29")
+					(reference "U706")
 					(unit 4)
 				)
@@
 		(on_board yes)
 		(dnp no)
-		(property "Reference" "R38"
+		(property "Reference" "R901"
 			(at 243.84 99.06 90)
 			(effects
@@
 			)
 		)
-		(property "Footprint" ""
+		(property "Footprint" "Resistor_SMD:R_0402_1005Metric"
 			(at 243.84 94.488 90)
 			(effects
@@
 			(project "6502sbc"
 				(path "/dc8636f6-e59e-4c75-ae27-408ad57a23de/78558388-3613-4012-b027-bd956c6e0596"
-					(reference "R38")
+					(reference "R901")
 					(unit 1)
 				)
@@
 		(on_board yes)
 		(dnp no)
-		(property "Reference" "D3"
+		(property "Reference" "D901"
 			(at 250.444 93.98 0)
 			(effects
@@
 			)
 		)
-		(property "Footprint" ""
+		(property "Footprint" "LED_SMD:LED_0402_1005Metric"
 			(at 254 92.71 0)
 			(effects
@@
 			(project "6502sbc"
 				(path "/dc8636f6-e59e-4c75-ae27-408ad57a23de/78558388-3613-4012-b027-bd956c6e0596"
-					(reference "D3")
+					(reference "D901")
 					(unit 1)
 				)
@@
 		(on_board yes)
 		(dnp no)
-		(property "Reference" "U2"
+		(property "Reference" "U110"
 			(at 70.612 148.336 0)
 			(effects
@@
 			(project "6502sbc"
 				(path "/dc8636f6-e59e-4c75-ae27-408ad57a23de/78558388-3613-4012-b027-bd956c6e0596"
-					(reference "U2")
+					(reference "U110")
 					(unit 2)
 				)
@@
 		(dnp no)
 		(fields_autoplaced yes)
-		(property "Reference" "U29"
+		(property "Reference" "U706"
 			(at 43.1717 39.37 0)
 			(effects
@@
 			(project "6502sbc"
 				(path "/dc8636f6-e59e-4c75-ae27-408ad57a23de/78558388-3613-4012-b027-bd956c6e0596"
-					(reference "U29")
+					(reference "U706")
 					(unit 3)
 				)
@@
 		(on_board yes)
 		(dnp no)
-		(property "Reference" "U9"
+		(property "Reference" "U507"
 			(at 70.612 130.048 0)
 			(effects
@@
 			(project "6502sbc"
 				(path "/dc8636f6-e59e-4c75-ae27-408ad57a23de/78558388-3613-4012-b027-bd956c6e0596"
-					(reference "U9")
+					(reference "U507")
 					(unit 2)
 				)
@@
 		(dnp no)
 		(fields_autoplaced yes)
-		(property "Reference" "U11"
+		(property "Reference" "U510"
 			(at 93.98 140.97 0)
 			(effects
@@
 			(project "6502sbc"
 				(path "/dc8636f6-e59e-4c75-ae27-408ad57a23de/78558388-3613-4012-b027-bd956c6e0596"
-					(reference "U11")
+					(reference "U510")
 					(unit 2)
 				)
@@
 		(dnp no)
 		(fields_autoplaced yes)
-		(property "Reference" "U29"
+		(property "Reference" "U706"
 			(at 43.1717 69.85 0)
 			(effects
@@
 			(project "6502sbc"
 				(path "/dc8636f6-e59e-4c75-ae27-408ad57a23de/78558388-3613-4012-b027-bd956c6e0596"
-					(reference "U29")
+					(reference "U706")
 					(unit 1)
 				)
@@
 		(on_board yes)
 		(dnp no)
-		(property "Reference" "#PWR0135"
+		(property "Reference" "#PWR0903"
 			(at 238.76 95.25 0)
 			(effects
@@
 			(project "6502sbc"
 				(path "/dc8636f6-e59e-4c75-ae27-408ad57a23de/78558388-3613-4012-b027-bd956c6e0596"
-					(reference "#PWR0135")
+					(reference "#PWR0903")
 					(unit 1)
 				)
@@
 		(dnp no)
 		(fields_autoplaced yes)
-		(property "Reference" "U5"
-			(at 134.62 153.67 0)
+		(property "Reference" "U106"
+			(at 134.62 154.94 0)
 			(effects
 				(font
@@
 		)
 		(property "Value" "SN74LS07"
-			(at 134.62 156.21 0)
+			(at 134.62 157.48 0)
 			(effects
 				(font
@@
 			(project "6502sbc"
 				(path "/dc8636f6-e59e-4c75-ae27-408ad57a23de/78558388-3613-4012-b027-bd956c6e0596"
-					(reference "U5")
+					(reference "U106")
 					(unit 6)
 				)
@@
 		(dnp no)
 		(fields_autoplaced yes)
-		(property "Reference" "U7"
+		(property "Reference" "U505"
 			(at 119.38 149.86 0)
 			(effects
@@
 			(project "6502sbc"
 				(path "/dc8636f6-e59e-4c75-ae27-408ad57a23de/78558388-3613-4012-b027-bd956c6e0596"
-					(reference "U7")
+					(reference "U505")
 					(unit 2)
 				)
@@
 		(dnp no)
 		(fields_autoplaced yes)
-		(property "Reference" "#PWR0134"
+		(property "Reference" "#PWR0902"
 			(at 227.33 86.36 0)
 			(effects
@@
 			(project "6502sbc"
 				(path "/dc8636f6-e59e-4c75-ae27-408ad57a23de/78558388-3613-4012-b027-bd956c6e0596"
-					(reference "#PWR0134")
+					(reference "#PWR0902")
 					(unit 1)
 				)
@@
 		(dnp no)
 		(fields_autoplaced yes)
-		(property "Reference" "#PWR0133"
+		(property "Reference" "#PWR0901"
 			(at 120.65 167.64 0)
 			(effects
@@
 			(project "6502sbc"
 				(path "/dc8636f6-e59e-4c75-ae27-408ad57a23de/78558388-3613-4012-b027-bd956c6e0596"
-					(reference "#PWR0133")
+					(reference "#PWR0901")
 					(unit 1)
 				)
@@
 		(dnp no)
 		(fields_autoplaced yes)
-		(property "Reference" "U2"
+		(property "Reference" "U110"
 			(at 217.1617 54.61 0)
 			(effects
@@
 			(project "6502sbc"
 				(path "/dc8636f6-e59e-4c75-ae27-408ad57a23de/78558388-3613-4012-b027-bd956c6e0596"
-					(reference "U2")
+					(reference "U110")
 					(unit 1)
 				)
@@
 	)
 	(symbol
+		(lib_name "SN74LS07_1")
 		(lib_id "74xx:SN74LS07")
 		(at 260.35 82.55 270)
@@
 		(dnp no)
 		(fields_autoplaced yes)
-		(property "Reference" "U5"
+		(property "Reference" "U106"
 			(at 267.97 82.55 0)
 			(effects
@@
 			(project "6502sbc"
 				(path "/dc8636f6-e59e-4c75-ae27-408ad57a23de/78558388-3613-4012-b027-bd956c6e0596"
-					(reference "U5")
+					(reference "U106")
 					(unit 3)
 				)
@@
 		(on_board yes)
 		(dnp no)
-		(property "Reference" "JP24"
+		(property "Reference" "JP901"
 			(at 77.978 138.938 0)
 			(effects
@@
 			)
 		)
-		(property "Footprint" ""
+		(property "Footprint" "Jumper:SolderJumper-2_P1.3mm_Bridged2Bar_Pad1.0x1.5mm"
 			(at 76.2 140.97 0)
 			(effects
@@
 			(project "6502sbc"
 				(path "/dc8636f6-e59e-4c75-ae27-408ad57a23de/78558388-3613-4012-b027-bd956c6e0596"
-					(reference "JP24")
+					(reference "JP901")
 					(unit 1)
 				)
@@
 		(dnp no)
 		(fields_autoplaced yes)
-		(property "Reference" "U23"
+		(property "Reference" "U503"
 			(at 87.63 96.5088 90)
 			(effects
@@
 			)
 		)
-		(property "Footprint" ""
+		(property "Footprint" "Package_SO:TSSOP-8_3x3mm_P0.65mm"
 			(at 80.01 99.06 0)
 			(effects
@@
 			(project "6502sbc"
 				(path "/dc8636f6-e59e-4c75-ae27-408ad57a23de/78558388-3613-4012-b027-bd956c6e0596"
-					(reference "U23")
+					(reference "U503")
 					(unit 2)
 				)
