File: hardware/6502sbc/6502sbc.kicad_sch (KiCad schematic)
At the start: 71 parts, among them J1 Conn_01x02_Pin, J2 Conn_01x02_Pin, J21 Clock input, U1 CD74HC4002M96, U2 74AHC08D-Q100J, U3 W65C02SxP, U4 74HC04, U49 74HC04, U5 SN74LS07, U53 74AHC2G00, U54 SN74CBT3245CDBR, U55 SN74CBT3245CDBR, U6 W65C22SxP

Commit message: Most footprints assigned
Parts:
- added U102, U103: 74HC74, Package_SO:SOIC-14_3.9x8.7mm_P1.27mm, symbol 74xx:74HC74
- C101: renamed from C1; footprint (none) -> Capacitor_SMD:C_0402_1005Metric
- C102: renamed from C2; footprint (none) -> Capacitor_SMD:C_0402_1005Metric
- C103: renamed from C3; footprint (none) -> Capacitor_SMD:C_0402_1005Metric
- C104: renamed from C4; footprint (none) -> Capacitor_SMD:C_0402_1005Metric
- C105: renamed from C70; footprint (none) -> Capacitor_SMD:C_0402_1005Metric
- C106: renamed from C69; footprint (none) -> Capacitor_SMD:C_0402_1005Metric
- D101: renamed from D15; footprint (none) -> LED_SMD:LED_0402_1005Metric
- JP101: renamed from JP33; footprint (none) -> Jumper:SolderJumper-2_P1.3mm_Bridged2Bar_Pad1.0x1.5mm
- JP102: renamed from JP4; footprint (none) -> Jumper:SolderJumper-3_P1.3mm_Bridged12_Pad1.0x1.5mm
- JP103: renamed from JP34; footprint (none) -> Jumper:SolderJumper-3_P1.3mm_Bridged12_Pad1.0x1.5mm
- JP104: renamed from JP1; footprint (none) -> Jumper:SolderJumper-3_P1.3mm_Bridged12_Pad1.0x1.5mm
- JP105: renamed from JP2; footprint (none) -> Jumper:SolderJumper-3_P1.3mm_Bridged12_Pad1.0x1.5mm
- JP106: renamed from JP3; footprint (none) -> Jumper:SolderJumper-3_P1.3mm_Bridged12_Pad1.0x1.5mm
- JP107: renamed from JP5; footprint (none) -> Jumper:SolderJumper-3_P1.3mm_Bridged12_Pad1.0x1.5mm
- JP108: renamed from JP6; footprint (none) -> Jumper:SolderJumper-3_P1.3mm_Bridged12_Pad1.0x1.5mm
- R101: renamed from R1; footprint (none) -> Resistor_SMD:R_0402_1005Metric
- R102: renamed from R2; footprint (none) -> Resistor_SMD:R_0402_1005Metric
- R103: renamed from R3; footprint (none) -> Resistor_SMD:R_0402_1005Metric
- R104: renamed from R4; footprint (none) -> Resistor_SMD:R_0402_1005Metric
- R105: renamed from R5; footprint (none) -> Resistor_SMD:R_0402_1005Metric
- R106: renamed from R130; footprint (none) -> Resistor_SMD:R_0402_1005Metric
- R107: renamed from R6; footprint (none) -> Resistor_SMD:R_0402_1005Metric
- R108: renamed from R131; footprint (none) -> Resistor_SMD:R_0402_1005Metric
- R109: renamed from R129; footprint (none) -> Resistor_SMD:R_0402_1005Metric
- R110: renamed from R104; footprint (none) -> Resistor_SMD:R_0402_1005Metric
- R111: renamed from R105; footprint (none) -> Resistor_SMD:R_0402_1005Metric
- R112: renamed from R106; footprint (none) -> Resistor_SMD:R_0402_1005Metric
- R113: renamed from R107; footprint (none) -> Resistor_SMD:R_0402_1005Metric
- R114: renamed from R108; footprint (none) -> Resistor_SMD:R_0402_1005Metric
- R115: renamed from R109; footprint (none) -> Resistor_SMD:R_0402_1005Metric
- R116: renamed from R110; footprint (none) -> Resistor_SMD:R_0402_1005Metric
- R117: renamed from R111; footprint (none) -> Resistor_SMD:R_0402_1005Metric
- R118: renamed from R112; footprint (none) -> Resistor_SMD:R_0402_1005Metric
- R119: renamed from R113; footprint (none) -> Resistor_SMD:R_0402_1005Metric
- R120: renamed from R114; footprint (none) -> Resistor_SMD:R_0402_1005Metric
- R121: renamed from R115; footprint (none) -> Resistor_SMD:R_0402_1005Metric
- R122: renamed from R116; footprint (none) -> Resistor_SMD:R_0402_1005Metric
- R123: renamed from R117; footprint (none) -> Resistor_SMD:R_0402_1005Metric
- R124: renamed from R118; footprint (none) -> Resistor_SMD:R_0402_1005Metric
- R125: renamed from R119; footprint (none) -> Resistor_SMD:R_0402_1005Metric
- R126: renamed from R96; footprint (none) -> Resistor_SMD:R_0402_1005Metric
- R127: renamed from R97; footprint (none) -> Resistor_SMD:R_0402_1005Metric
- R128: renamed from R98; footprint (none) -> Resistor_SMD:R_0402_1005Metric
- R129: renamed from R99; footprint (none) -> Resistor_SMD:R_0402_1005Metric
- R130: renamed from R100; footprint (none) -> Resistor_SMD:R_0402_1005Metric
- R131: renamed from R101; footprint (none) -> Resistor_SMD:R_0402_1005Metric
- R132: renamed from R102; footprint (none) -> Resistor_SMD:R_0402_1005Metric
- R133: renamed from R103; footprint (none) -> Resistor_SMD:R_0402_1005Metric
- R134: renamed from R78; footprint (none) -> Resistor_SMD:R_0402_1005Metric
- R135: renamed from R128; footprint (none) -> Resistor_SMD:R_0402_1005Metric
- R136: renamed from R127; footprint (none) -> Resistor_SMD:R_0402_1005Metric
- TP101: renamed from TP11; footprint (none) -> TestPoint:TestPoint_Pad_D2.5mm
- TP102: renamed from TP1; footprint (none) -> TestPoint:TestPoint_Pad_D1.5mm
- TP103: renamed from TP12; footprint (none) -> TestPoint:TestPoint_Pad_D2.5mm
- TP104: renamed from TP8; footprint (none) -> TestPoint:TestPoint_Pad_D1.5mm
- TP105: renamed from TP10; footprint (none) -> TestPoint:TestPoint_Pad_D1.5mm
- TP106: renamed from TP2; footprint (none) -> TestPoint:TestPoint_Pad_D1.5mm
- TP107: renamed from TP9; footprint (none) -> TestPoint:TestPoint_Pad_D1.5mm
- U107: renamed from U53; footprint (none) -> Package_SO:TSSOP-8_3x3mm_P0.65mm
- U111: renamed from U54; footprint (none) -> Package_SO:SSOP-20_5.3x7.2mm_P0.65mm
- U112: renamed from U55; footprint (none) -> Package_SO:SSOP-20_5.3x7.2mm_P0.65mm
- renumbered J21 to J101, J1 to J102, J2 to J103, U4 to U101, U3 to U104, U1 to U105, U5 to U106, U6 to U108, U49 to U109, U2 to U110
Connections:
- net +5V: now also U102.1 (~{R}), U102.13 (~{R}), U103.1 (~{R}), U103.13 (~{R})
- net PHI2: now also U102.11 (C), U102.3 (C), U103.11 (C), U103.3 (C)
- net RESB: now also U102.10 (~{S}), U102.4 (~{S}), U103.10 (~{S}), U103.4 (~{S})
- net ~{IRQ}: now also U102.12 (D); no longer U104.4 (~{IRQ})
- net ~{NMI}: now also U103.12 (D); no longer U104.6 (~{NMI})
- new net: U103.2 (D), U103.9 (Q)
- new net: U102.2 (D), U102.9 (Q)
- new net ~{IRQ_SYNC}: U102.5 (Q), U104.4 (~{IRQ})
- new net ~{NMI_SYNC}: U103.5 (Q), U104.6 (~{NMI})
- no-connect marks 4 -> 8
Other:
- sheet DMA Peripheral Interface ports: added RESB; removed none
- sheet High-Memory Address Decode ports: added A4; removed none
- sheet Privileges & Exception Handling ports: added SYNC; removed none
- note added: "Interrupt Synchronization"
- moved on the sheet: C101, C102, J101, J102, J103, R101, R102, R103, R104, R105, R107, R108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

Commit message: Ready to begin pcb layout
Parts:
- removed U104: W65C02SxP, Package_LCC:PLCC-44, symbol PCM_65xx-library:W65C02SxP
- removed U108: W65C22SxP, Package_LCC:PLCC-44, symbol PCM_65xx-library:W65C22SxP
- added TP108: phi2O, TestPoint:TestPoint_Pad_D1.5mm, symbol Connector:TestPoint
- added TP109: phi1, TestPoint:TestPoint_Pad_D1.5mm, symbol Connector:TestPoint
- added U104: W65C02SxPL, Package_LCC:PLCC-44, symbol PCM_65xx-library:W65C02SxPL
- added U108: W65C22SxPL, Package_LCC:PLCC-44, symbol PCM_65xx-library:W65C22SxPL
Connections:
- net +5V: now also U104.37 (VDD), U104.9 (VDD), U108.21 (VDD)
- net A0: now also U108.42 (RS0)
- net A1: now also U108.41 (RS1)
- net A2: now also U108.40 (RS2)
- net A3: now also U108.39 (RS3)
- net Character IO/LCDEN: now also U108.13 (PB2)
- net Character IO/LCDSEL0: now also U108.10 (PB0)
- net Character IO/LCDSEL1: now also U108.12 (PB1)
- net Character IO/LCD_RS: now also U108.14 (PB3)
- net Character IO/PA0: now also U108.2 (PA0)
- net Character IO/PA1: now also U108.3 (PA1)
- net Character IO/PA2: now also U108.4 (PA2)
- net Character IO/PA3: now also U108.5 (PA3)
- net Character IO/PA4: now also U108.6 (PA4)
- net Character IO/PA5: now also U108.7 (PA5)
- net Character IO/PA6: now also U108.8 (PA6)
- net Character IO/PA7: now also U108.9 (PA7)
- net Character IO/~{DATA_READY}: now also U108.44 (CA1)
- net Character IO/~{DATA_TAKEN}: now also U108.43 (CA2)
- net D0: now also U108.36 (D0)
- net D1: now also U108.35 (D1)
- net D2: now also U108.34 (D2)
- net D3: now also U108.32 (D3)
- net D4: now also U108.31 (D4)
- net D5: now also U108.30 (D5)
- net D6: now also U108.29 (D6)
- net D7: now also U108.28 (D7)
- net GND: now also U104.1 (VSS), U104.23 (VSS), U104.24 (VSS), U108.1 (VSS)
- net IO_CMD: now also U108.16 (PB5)
- net NMI_TIMER: now also U108.18 (PB7)
- net PHI2: now also U104.41 (ϕ0)
- net RDY: now also U104.3 (RDY)
- net RESB: now also U104.44 (~{RES}), U108.37 (~{RES})
- net R~{W}: now also U108.24 (R/~{W})
- net SYNC: now also U104.8 (SYNC)
- net VIACLK: now also U108.27 (ϕ2)
- net VIA_CS1: now also U108.26 (CS1)
- net VIA_~{CS2}: now also U108.25 (~{CS2})
- net ~{IRQ_SYNC}: now also U104.5 (~{IRQ})
- net ~{ML}: now also U104.6 (~{ML})
- net ~{NMI_SYNC}: now also U104.7 (~{NMI})
- net ~{UMINH}: now also U108.15 (PB4)
- net ~{VPB}: now also U104.2 (~{VP})
- net ~{WRITBANKEN}: now also U108.17 (PB6)
- net at R111.1: now also U104.11 (A1)
- net at R132.1: now also U104.30 (D6)
- net at R112.1: now also U104.13 (A2)
- net at R124.1: now also U104.27 (A14)
- net at R101.2: now also U104.42 (~{SO})
- net at R125.1: now also U104.28 (A15)
- net at R110.1: now also U104.10 (A0)
- net at U106.9: now also U108.23 (~{IRQ})
- net at R113.1: now also U104.14 (A3)
- net at R114.1: now also U104.15 (A4)
- net at R115.1: now also U104.16 (A5)
- net at R116.1: now also U104.17 (A6)
- net at R117.1: now also U104.18 (A7)
- net at R118.1: now also U104.19 (A8)
- net at R119.1: now also U104.20 (A9)
- net at R120.1: now also U104.21 (A10)
- net at R121.1: now also U104.22 (A11)
- net at R122.1: now also U104.25 (A12)
- net at R123.1: now also U104.26 (A13)
- net at R133.1: now also U104.29 (D7)
- net at R131.1: now also U104.31 (D5)
- net at R130.1: now also U104.32 (D4)
- net at R129.1: now also U104.33 (D3)
- net at R128.1: now also U104.34 (D2)
- net at R127.1: now also U104.35 (D1)
- net at R126.1: now also U104.36 (D0)
- net at R108.2: now also U104.38 (R/~{W})
- net at R102.2: now also U104.40 (BE)
- new net: TP109.1, U104.4 (ϕ1)
- new net: TP108.1, U104.43 (ϕ2O)
- no-connect marks 8 -> 6
Other:
- moved on the sheet: R108, TP102
