File: hardware/6502sbc/char_io.kicad_sch (KiCad schematic)
At the start: 29 parts, among them J24 KMDGX-6S-BS, J29 Parallel LCD, J30 Parallel LCD, J31 Parallel LCD, J32 Parallel LCD, Q1 2N7002K, U37 74HC04, U38 74HC595, U39 74HC193, U40 74ACT139

Commit message: Preliminary schematic
Parts:
- renumbered C42 to C38, C43 to C39, C38 to C40, C39 to C41, C40 to C42, C41 to C43, J29 to J28, J31 to J29, J32 to J31, J24 to J32, JP23 to JP25, JP29 to JP26, JP24 to JP27, JP30 to JP28, JP31 to JP29, JP27 to JP30, JP28 to JP31, RV4 to RV2, RV5 to RV3, RV2 to RV4, RV3 to RV5, U40 to U36

Commit message: Schematic is nearly done
Parts:
- added C77, C79, C80, C81, C82: 1u, symbol Device:C_Polarized
- added C78: .1u, symbol Device:C_Polarized
- C41: value .01u -> u
- C42, C43: value .01u -> .1u
- U37: footprint (none) -> Package_SO:SOIC-14_3.9x8.7mm_P1.27mm; t_pd (ns) (none) -> 19
Connections:
- net +5V: now also C77.1, C78.1, C79.1, C80.1, C81.1, C82.1
- net GND: now also C77.2, C78.2, C79.2, C80.2, C81.2, C82.2

Commit message: Most footprints assigned
Parts:
- removed C77, C79, C80, C81, C82: 1u, symbol Device:C_Polarized
- removed C78: .1u, symbol Device:C_Polarized
- added C1003, C1004, C1005, C1006, C1009: 10u, Capacitor_SMD:C_0402_1005Metric, symbol Device:C
- added C1012: 0.1u, Capacitor_SMD:C_0402_1005Metric, symbol Device:C
- C1001: renamed from C38; footprint (none) -> Capacitor_SMD:C_0402_1005Metric
- C1002: renamed from C39; footprint (none) -> Capacitor_SMD:C_0402_1005Metric
- C1007: renamed from C40; footprint (none) -> Capacitor_SMD:C_0402_1005Metric
- C1008: renamed from C41; value u -> 1u; footprint (none) -> Capacitor_SMD:C_0402_1005Metric
- C1010: renamed from C42; footprint (none) -> Capacitor_SMD:C_0402_1005Metric
- C1011: renamed from C43; footprint (none) -> Capacitor_SMD:C_0402_1005Metric
- JP1001: renamed from JP25; footprint (none) -> Jumper:SolderJumper-2_P1.3mm_Bridged2Bar_Pad1.0x1.5mm
- JP1002: renamed from JP26; footprint (none) -> Jumper:SolderJumper-2_P1.3mm_Bridged2Bar_Pad1.0x1.5mm
- JP1003: renamed from JP27; footprint (none) -> Jumper:SolderJumper-2_P1.3mm_Bridged2Bar_Pad1.0x1.5mm
- JP1004: renamed from JP28; footprint (none) -> Jumper:SolderJumper-2_P1.3mm_Bridged2Bar_Pad1.0x1.5mm
- JP1005: renamed from JP29; footprint (none) -> Jumper:SolderJumper-2_P1.3mm_Bridged2Bar_Pad1.0x1.5mm
- JP1006: renamed from JP30; footprint (none) -> Jumper:SolderJumper-3_P1.3mm_Bridged12_Pad1.0x1.5mm
- JP1007: renamed from JP31; footprint (none) -> Jumper:SolderJumper-3_P1.3mm_Bridged12_Pad1.0x1.5mm
- R1001: renamed from R39; footprint (none) -> Resistor_SMD:R_0402_1005Metric
- R1002: renamed from R40; footprint (none) -> Resistor_SMD:R_0402_1005Metric
- U1001: renamed from U36; footprint (none) -> Package_SO:TSSOP-16_4.4x5mm_P0.65mm
- U1003: renamed from U38; footprint (none) -> Package_SO:SOIC-16_3.9x9.9mm_P1.27mm
- U1004: renamed from U39; footprint (none) -> Package_SO:TSSOP-16_4.4x5mm_P0.65mm
- renumbered J28 to J1001, J29 to J1002, J30 to J1003, J31 to J1004, J32 to J1005, Q1 to Q1001, RV2 to RV1001, RV3 to RV1002, RV4 to RV1003, RV5 to RV1004, U37 to U1002
Connections:
- net +5V: now also C1003.1, C1004.1, C1005.1, C1006.1, C1009.1, C1012.1
- net GND: now also C1003.2, C1004.2, C1005.2, C1006.2, C1009.2, C1012.2

Commit message: Ready to begin pcb layout
Parts:
- added J1006: KMDGX-6S-BS, KMDGX6SBS, symbol PS2 Connector:KMDGX-6S-BS
- J1005: now left out of the parts list
Connections:
- net +5V: now also J1006.5
- net GND: now also J1006.3, J1006.MH1, J1006.MH2, J1006.MH3
- net KEY_CLK: now also J1006.6
- net KEY_DAT: now also J1006.1
- no-connect marks 13 -> 15
Other:
- note added: "(Actual Connector)"
- moved on the sheet: C1007, C1008
