File: hardware/6502sbc/power.kicad_sch (KiCad schematic)
At the start: 15 parts, among them J16 +5VDC, J17 Clock input, U19 74AHC2G00, U2 SN74LS07, U3 LD1117S33TR_SOT223, U4 LD1117STR

Commit message: Preliminary schematic
Parts:
- added D12, D13, D14: LED, symbol Device:LED
- added R75, R76: 470, symbol Device:R
- added R77: 510, symbol Device:R
- renumbered C3 to C25, C2 to C26, C1 to C27, C4 to C28, C7 to C29, J16 to J20, J17 to J21, JP4 to JP19, JP3 to JP20, R1 to R27, U4 to U21, U3 to U22, U19 to U23, U2 to U5
Connections:
- net +3V3: now also R76.1, R77.1
- net GND: now also D12.1 (K), D13.1 (K), D14.1 (K)
- net Vadj renamed +2V8
- net +2V8: now also R75.1
- new net: D14.2 (A), R77.2
- new net: D12.2 (A), R75.2
- new net: D13.2 (A), R76.2
Other:
- note added: "3V3 Supply ON"
- note added: "5V Supply"
- note added: "SRAM Data Overvolt Protection Supply ON"

Commit message: Schematic is nearly done
Parts:
- removed J21: Clock input, symbol Connector:Conn_01x02_Pin
- added C100, C101, C102, C103, C104, C105, C93, C94, C97, C98, C99: .1u, symbol Device:C_Polarized
- added C106, C107, C95, C96: 1u, symbol Device:C_Polarized
- added U1, U9: CD74HC4002M96, Package_SO:SOIC-14_3.9x8.7mm_P1.27mm, symbol custom:_1
- added U10, U11, U8: 74AHC2G32DP, Package_SO:TSSOP-8_3x3mm_P0.65mm, symbol 74xGxx:74LVC2G32
- added U2: 74AHC08D-Q100J, Package_SO:SOIC-14_3.9x8.7mm_P1.27mm, symbol 74xx:74LS08
- added U4: 74HC04, Package_SO:SOIC-14_3.9x8.7mm_P1.27mm, symbol 74xx:74HC04
- added U53: 74AHC2G00, symbol 74xGxx:74AHC2G00
- added U7: 74HC73D, Package_SO:SOIC-14_3.9x8.7mm_P1.27mm, symbol 74xx:74LS73
- U5: footprint (none) -> Package_SO:SOIC-14_3.9x8.7mm_P1.27mm; t_pd (ns) (none) -> 30
Connections:
- net +3V3: now also C107.1, C96.1
- net +5V: now also U23.8 (VCC), U5.14 (VCC), C100.1, C101.1, C102.1, C103.1, C104.1, C105.1, C106.1, C93.1, C94.1, C95.1, C97.1, C98.1, C99.1, U1.14 (VCC), U10.8 (VCC), U11.8 (VCC), U2.14 (VCC), U4.14 (VCC), U53.8 (VCC), U7.4 (VCC), U8.8 (VCC), U9.14 (VCC)
- net GND: now also U23.4 (GND), U5.7 (GND), C100.2, C101.2, C102.2, C103.2, C104.2, C105.2, C106.2, C107.2, C93.2, C94.2, C95.2, C96.2, C97.2, C98.2, C99.2, U1.7 (GND), U10.4 (GND), U11.4 (GND), U2.7 (GND), U4.7 (GND), U53.4 (GND), U7.11 (GND), U8.4 (GND), U9.7 (GND)
Other:
- moved on the sheet: C25, C26, C27, C28, C29, D12, D13, D14, J20, JP19, JP20, R27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

Commit message: Most footprints assigned
Parts:
- removed C100, C101, C102, C103, C104, C105, C93, C94, C97, C98, C99: .1u, symbol Device:C_Polarized
- removed C106, C107, C95, C96: 1u, symbol Device:C_Polarized
- removed C27, C28: 10u, symbol Device:C_Polarized
- removed C29: 4.7u, symbol Device:C_Polarized
- removed JP19, JP20: Jumper_2_Small_Bridged, symbol Jumper:Jumper_2_Small_Bridged
- removed U5: SN74LS07, Package_SO:SOIC-14_3.9x8.7mm_P1.27mm, symbol 74xx:SN74LS07
- added C503, C504, C505, C506, C507, C510, C511: 10u, Capacitor_SMD:C_0402_1005Metric, symbol Device:C
- added C508, C509, C512, C513, C515, C517, C518, C519, C520, C521, C522: 0.1u, Capacitor_SMD:C_0402_1005Metric, symbol Device:C
- added C514, C516: .1u, Capacitor_SMD:C_0402_1005Metric, symbol Device:C
- added TP501, TP502: TestPoint, TestPoint:TestPoint_Pad_D2.5mm, symbol Connector:TestPoint
- added U102, U103: 74HC74, Package_SO:SOIC-14_3.9x8.7mm_P1.27mm, symbol 74xx:74HC74
- added U106: SN74LS07, Package_SO:SOIC-14_3.9x8.7mm_P1.27mm, symbol 74xx:SN74LS07
- C501: renamed from C25; footprint (none) -> Capacitor_SMD:C_0402_1005Metric
- C502: renamed from C26; footprint (none) -> Capacitor_SMD:C_0402_1005Metric
- D501: renamed from D12; footprint (none) -> LED_SMD:LED_0402_1005Metric
- D502: renamed from D13; footprint (none) -> LED_SMD:LED_0402_1005Metric
- D503: renamed from D14; footprint (none) -> LED_SMD:LED_0402_1005Metric
- R501: renamed from R75; footprint (none) -> Resistor_SMD:R_0402_1005Metric
- R502: renamed from R76; footprint (none) -> Resistor_SMD:R_0402_1005Metric
- R503: renamed from R27; footprint (none) -> Resistor_SMD:R_0402_1005Metric
- R504: renamed from R77; footprint (none) -> Resistor_SMD:R_0402_1005Metric
- U107: renamed from U53; footprint (none) -> Package_SO:TSSOP-8_3x3mm_P0.65mm
- U503: renamed from U23; footprint (none) -> Package_SO:TSSOP-8_3x3mm_P0.65mm
- renumbered J20 to J501, RV1 to RV501, U4 to U101, U1 to U105, U2 to U110, U21 to U501, U22 to U502, U7 to U505, U9 to U507, U10 to U508, U8 to U509, U11 to U510
Connections:
- net +2V8: now also R503.1, U501.2 (VO), C504.1, TP502.1
- net +3V3: now also U502.2 (VO), C503.1, C507.1, C511.1, TP501.1
- net +5V: now also C505.1, C506.1, C508.1, C509.1, C510.1, C512.1, C513.1, C514.1, C515.1, C516.1, C517.1, C518.1, C519.1, C520.1, C521.1, C522.1, U102.14 (VCC), U103.14 (VCC), U106.14 (VCC)
- net GND: now also C503.2, C504.2, C505.2, C506.2, C507.2, C508.2, C509.2, C510.2, C511.2, C512.2, C513.2, C514.2, C515.2, C516.2, C517.2, C518.2, C519.2, C520.2, C521.2, C522.2, U102.7 (GND), U103.7 (GND), U106.7 (GND)
