File: kicad_project/Hombrew6502Project/Hombrew6502Project.kicad_pcb (KiCad board)
At the start: 2 copper layers, 353 parts, among them J1006 KMDGX-6S-BS, Q1001 2N7002K, U1001 74ACT139, U1002 74HC04, U1003 74HC595, U1004 74HC193, U101 74HC04, U102 74HC74, U103 74HC74, U104 W65C02SxP, U105 CD74HC4002M96, U106 SN74LS07, U107 74AHC2G00, U108 W65C22SxP, U109 74HC04, U110 74AHC08D-Q100J, U111 SN74CBT3245CDBR, U112 SN74CBT3245CDBR, U201 SN74LS07, U202 CY7C146-25JC, U203 PIC16F15385-xPT, U301 TXS0108EPW, U303 74FCT521ATSOG8, U304 74ACT139, U305 74LVC244APW, U307 74LVC244APW, U309 74ACT139, U311 74LVC244APW, U401 74HCT125D, U402 M95512-Axxx-MF, U501 LD1117STR, U502 LD1117S33TR_SOT223, U503 74AHC2G00, U505 74HC73D, U507 CD74HC4002M96, U508 74AHC2G32DP, U509 74AHC2G32DP, U510 74AHC2G32DP, U701 74AHC2G00, U702 74AHC2G00, U703 74AHC08D-Q100J, U704 CD74HC4002M96, U705 CD74HC4002M96, U706 74AHC08D-Q100J, U801 74ACT139, U802 SN74ABT574APWR, U803 SN74ABT574APWR, U804 SN74ABT574APWR, U805 SN74ABT574APWR, U806 SN74ABT574APWR, Y201 NOPOP

Commit message: Some connector changes
Parts:
- added REF**: PinSocket_2x05_P2.54mm_Vertical, Connector_PinSocket_2.54mm:PinSocket_2x05_P2.54mm_Vertical, F.Cu at (268.0, 34.0)
- moved J1006 245.8 mm to (-20.3, 138.3)
- moved Q1001 226.3 mm to (-34.7, 140.3)
- moved R1001 218.1 mm to (-40.0, 114.5)
- moved U1002 216.7 mm to (-43.0, 129.0)
- moved R1002 215.2 mm to (-21.5, 148.0)
- moved C302 203.9 mm to (210.5, 273.5)
- moved C303 203.9 mm to (210.5, 275.5)
- moved C304 203.9 mm to (210.5, 277.4)
- moved C305 203.9 mm to (210.5, 279.4)
- moved C307 203.9 mm to (210.5, 283.4)
- moved C306 203.9 mm to (210.5, 281.4)
- moved C308 203.9 mm to (210.5, 285.3)
- moved JP1006 203.0 mm to (-8.80, 149.0)
- moved U1003 191.2 mm to (-23.0, 98.7)
- moved U1001 189.4 mm to (-23.0, 121.5)
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Other:
- board text added: "Peripheral i/o"
- board text added: "SRAM BOARD"

Commit message: footprint assignments and separate project for RAM board
Parts:
- removed C301, C304: 10u, Capacitor_SMD:C_0402_1005Metric
- removed C302, C309, C316, C321: 1u, Capacitor_SMD:C_0402_1005Metric
- removed C303, C305, C306, C307, C310, C312, C314, C317, C322, C324, C326, C328: .01u, Capacitor_SMD:C_0402_1005Metric
- removed C308, C311, C313, C315, C318, C319, C320, C323, C325, C327, C329: .1u, Capacitor_SMD:C_0402_1005Metric
- removed D301, D305: LED, LED_SMD:LED_0402_1005Metric
- removed D302, D303, D304, D306, D307, D308, D309: BAT54CDW, Package_TO_SOT_SMD:SOT-363_SC-70-6
- removed JP301: Jumper_2_Small_Open, Jumper:SolderJumper-2_P1.3mm_Open_Pad1.0x1.5mm
- removed R309, R310, R311, R312, R313, R314, R315, R316: 33, Resistor_SMD:R_0402_1005Metric
- removed R317, R343: 470, Resistor_SMD:R_0402_1005Metric
- removed R318, R319, R320, R321, R322, R323, R324, R325, R327, R328, R329, R330, R331, R332, R333, R334, R335, R336, R337, R338, R339, R340, R341, R342, R344, R345, R346, R347, R348, R349, R350, R351: 100, Resistor_SMD:R_0402_1005Metric
- removed R326: 10K, Resistor_SMD:R_0402_1005Metric
- removed REF**: PinSocket_2x05_P2.54mm_Vertical, Connector_PinSocket_2.54mm:PinSocket_2x05_P2.54mm_Vertical
- removed RN301: R_Network08_US, Resistor_THT:R_Array_SIP9
- removed TP601, TP602, TP603, TP604: TestPoint, TestPoint:TestPoint_Pad_D1.5mm
- removed U301: TXS0108EPW, Package_SO:TSSOP-20_4.4x6.5mm_P0.65mm
- removed U302, U306, U308, U310: ~, Package_SO:TSOP-II-44_10.16x18.41mm_P0.8mm
- removed U303: 74FCT521ATSOG8, Package_SO:SOIC-20W_7.5x12.8mm_P1.27mm
- removed U304, U309: 74ACT139, Package_SO:TSSOP-16_4.4x5mm_P0.65mm
- removed U305, U307, U311: 74LVC244APW, Package_SO:TSSOP-20_4.4x6.5mm_P0.65mm
- added C523: 10u, Capacitor_SMD:C_0402_1005Metric, F.Cu at (92.5, 365.5)
- added J1001: Parallel LCD, Connector_IDC:IDC-Header_2x08_P2.54mm_Vertical_SMD, F.Cu at (-45.4, 235.9)
- added J1002: Parallel LCD, Connector_IDC:IDC-Header_2x08_P2.54mm_Vertical_SMD, F.Cu at (-30.7, 235.9)
- added J1003: Parallel LCD, Connector_IDC:IDC-Header_2x08_P2.54mm_Vertical_SMD, F.Cu at (-16.1, 235.9)
- added J1004: Parallel LCD, Connector_IDC:IDC-Header_2x08_P2.54mm_Vertical_SMD, F.Cu at (-1.41, 235.9)
- added J101: Conn_02x02_Odd_Even, Connector_PinHeader_2.54mm:PinHeader_2x02_P2.54mm_Vertical_SMD, F.Cu at (95.4, 311.1)
- added J104: Conn_02x02_Odd_Even, Connector_PinHeader_2.54mm:PinHeader_2x02_P2.54mm_Vertical_SMD, F.Cu at (95.4, 318.2)
- added J201: ICSP Header, Connector_PinHeader_2.54mm:PinHeader_1x06_P2.54mm_Vertical, F.Cu at (25.3, 355.9)
- added J202: Conn_02x05_Odd_Even, Connector_PinHeader_2.54mm:PinHeader_2x05_P2.54mm_Vertical_SMD, F.Cu at (30.3, 342.4)
- added J203: Conn_02x05_Odd_Even, Connector_PinHeader_2.54mm:PinHeader_2x05_P2.54mm_Vertical_SMD, F.Cu at (45.0, 342.4)
- added J204: I2C, Connector_PinHeader_2.54mm:PinHeader_1x05_P2.54mm_Vertical, F.Cu at (29.9, 355.9)
- added J205: Conn_02x05_Odd_Even, Connector_PinHeader_2.54mm:PinHeader_2x05_P2.54mm_Vertical_SMD, F.Cu at (59.6, 342.4)
- added J206: Conn_02x05_Odd_Even, Connector_PinHeader_2.54mm:PinHeader_2x05_P2.54mm_Vertical_SMD, F.Cu at (74.3, 342.4)
- added J210: UART, Connector:FanPinHeader_1x03_P2.54mm_Vertical, F.Cu at (34.4, 357.1)
- added J301: Conn_02x16_Odd_Even, Connector_PinHeader_2.54mm:PinHeader_2x16_P2.54mm_Vertical_SMD, F.Cu at (29.4, 307.9)
- added J302: Conn_02x16_Odd_Even, Connector_PinHeader_2.54mm:PinHeader_2x16_P2.54mm_Vertical_SMD, F.Cu at (42.2, 307.9)
- added J402: Micro_SD_Card, Connector_Card:microSD_HC_Wuerth_693072010801, F.Cu at (92.2, 339.1)
- added J403: Conn_02x03_Odd_Even, Connector_PinHeader_2.54mm:PinHeader_2x03_P2.54mm_Vertical_SMD, F.Cu at (90.0, 352.9)
- added J501: +5VDC, Connector_PinHeader_2.54mm:PinHeader_1x02_P2.54mm_Vertical, F.Cu at (85.9, 362.1)
- added JP109: Jumper_2_Small_Bridged, Jumper:SolderJumper-2_P1.3mm_Bridged2Bar_Pad1.0x1.5mm, F.Cu at (104.0, 309.3)
- added R505: 100, Resistor_SMD:R_0402_1005Metric, F.Cu at (89.6, 365.5)
- added RV1001: 10k, Potentiometer_SMD:Potentiometer_Bourns_TC33X_Vertical, F.Cu at (92.2, 288.9)
- added RV1002: 10k, Potentiometer_SMD:Potentiometer_Bourns_TC33X_Vertical, F.Cu at (92.2, 293.6)
- added RV1003: 10k, Potentiometer_SMD:Potentiometer_Bourns_TC33X_Vertical, F.Cu at (92.2, 298.4)
- added RV1004: 10k, Potentiometer_SMD:Potentiometer_Bourns_TC33X_Vertical, F.Cu at (92.2, 303.1)
- added RV501: 300, Potentiometer_SMD:Potentiometer_Bourns_TC33X_Vertical, F.Cu at (91.3, 362.1)
- added TP108: phi2O, TestPoint:TestPoint_Pad_D1.5mm, F.Cu at (18.5, 33.0)
- added TP109: phi1, TestPoint:TestPoint_Pad_D1.5mm, F.Cu at (13.0, 31.5)
- R301, R302, R303, R304, R305, R306, R307, R308: value 100 -> 0
- U104: value W65C02SxP -> W65C02SxPL
- U108: value W65C22SxP -> W65C22SxPL
- moved U802 104.8 mm to (-30.0, 205.0), turned to 90 degrees
- moved U108 34.2 mm to (-5.00, 87.0), turned to 90 degrees
- moved U104 0.45 mm to (16.7, 47.1)
Connections:
- JP201 pad 2: /DMA Peripheral Interface/DMA Peripheral Interface Module/6502_DMA_~{CS} -> /~{DMA_CS}
- JP202 pad 1: /DMA Peripheral Interface/DMA Peripheral Interface Module/6502_DMA_~{CS} -> /~{DMA_CS}
- U104 pad 1: /~{VPB} -> GND
- U104 pad 10: Net-(U104-A1) -> Net-(U104-A0)
- U104 pad 11: Net-(U104-A2) -> Net-(U104-A1)
- U104 pad 12: Net-(U104-A3) -> unconnected-(U104-nc-Pad12)
- U104 pad 13: Net-(U104-A4) -> Net-(U104-A2)
- U104 pad 14: Net-(U104-A5) -> Net-(U104-A3)
- U104 pad 15: Net-(U104-A6) -> Net-(U104-A4)
- U104 pad 16: Net-(U104-A7) -> Net-(U104-A5)
- U104 pad 17: Net-(U104-A8) -> Net-(U104-A6)
- U104 pad 18: Net-(U104-A9) -> Net-(U104-A7)
- U104 pad 19: Net-(U104-A10) -> Net-(U104-A8)
- U104 pad 2: /RDY -> /~{VPB}
- U104 pad 20: Net-(U104-A11) -> Net-(U104-A9)
- U104 pad 21: GND -> Net-(U104-A10)
- U104 pad 22: Net-(U104-A12) -> Net-(U104-A11)
- U104 pad 23: Net-(U104-A13) -> GND
- U104 pad 24: Net-(U104-A14) -> GND
- U104 pad 25: Net-(U104-A15) -> Net-(U104-A12)
- U104 pad 26: Net-(U104-D7) -> Net-(U104-A13)
- U104 pad 27: Net-(U104-D6) -> Net-(U104-A14)
- U104 pad 28: Net-(U104-D5) -> Net-(U104-A15)
- U104 pad 29: Net-(U104-D4) -> Net-(U104-D7)
- U104 pad 3: unconnected-(U104-ϕ1-Pad3) -> /RDY
- U104 pad 30: Net-(U104-D3) -> Net-(U104-D6)
- U104 pad 31: Net-(U104-D2) -> Net-(U104-D5)
- U104 pad 32: Net-(U104-D1) -> Net-(U104-D4)
- U104 pad 33: Net-(U104-D0) -> Net-(U104-D3)
- U104 pad 34: Net-(U104-R/~{W}) -> Net-(U104-D2)
- U104 pad 35: unconnected-(U104-nc-Pad35) -> Net-(U104-D1)
- U104 pad 36: Net-(U104-BE) -> Net-(U104-D0)
- U104 pad 37: PHI2 -> +5V
- U104 pad 38: Net-(U104-~{SO}) -> Net-(U104-R/~{W})
- U104 pad 4: /~{IRQ_SYNC} -> Net-(U104-ϕ1)
- U104 pad 40: RESB -> Net-(U104-BE)
- U104 pad 41: (no net) -> PHI2_CPU
- U104 pad 42: (no net) -> Net-(U104-~{SO})
- U104 pad 43: (no net) -> Net-(U104-ϕ2O)
- U104 pad 44: (no net) -> RESB
- U104 pad 5: /~{ML} -> /~{IRQ_SYNC}
- U104 pad 6: /~{NMI_SYNC} -> /~{ML}
- U104 pad 7: /SYNC -> /~{NMI_SYNC}
- U104 pad 8: +5V -> /SYNC
- U104 pad 9: Net-(U104-A0) -> +5V
- U108 pad 11: /Character IO/LCDSEL1 -> unconnected-(U108-nc-Pad11)
- U108 pad 12: /Character IO/LCDEN -> /Character IO/LCDSEL1
- U108 pad 13: /Character IO/LCD_RS -> /Character IO/LCDEN
- U108 pad 14: /~{UMINH} -> /Character IO/LCD_RS
- U108 pad 15: /IO_CMD -> /~{UMINH}
- U108 pad 16: /~{WRITBANKEN} -> /IO_CMD
- U108 pad 17: /NMI_TIMER -> /~{WRITBANKEN}
- U108 pad 18: unconnected-(U108-CB1-Pad18) -> /NMI_TIMER
- U108 pad 20: +5V -> unconnected-(U108-CB2-Pad20)
- U108 pad 21: Net-(U108-~{IRQ}) -> +5V
- U108 pad 22: /R~{W} -> unconnected-(U108-nc-Pad22)
- U108 pad 23: /VIA_~{CS2} -> Net-(U108-~{IRQ})
- U108 pad 24: /VIA_CS1 -> /R~{W}
- U108 pad 25: /VIACLK -> /VIA_~{CS2}
- U108 pad 26: /D7 -> /VIA_CS1
- U108 pad 27: /D6 -> /VIACLK
- U108 pad 28: /D5 -> /D7
- U108 pad 29: /D4 -> /D6
- U108 pad 30: /D3 -> /D5
- U108 pad 31: /D2 -> /D4
- U108 pad 32: /D1 -> /D3
- U108 pad 33: /D0 -> unconnected-(U108-nc-Pad33)
- U108 pad 34: RESB -> /D2
- U108 pad 35: /A3 -> /D1
- U108 pad 36: /A2 -> /D0
- U108 pad 37: /A1 -> RESB
- U108 pad 38: /A0 -> unconnected-(U108-nc-Pad38)
- U108 pad 39: /Character IO/~{DATA_TAKEN} -> /A3
- U108 pad 40: /Character IO/~{DATA_READY} -> /A2
- U108 pad 41: (no net) -> /A1
- U108 pad 42: (no net) -> /A0
- U108 pad 43: (no net) -> /Character IO/~{DATA_TAKEN}
- U108 pad 44: (no net) -> /Character IO/~{DATA_READY}
- U201 pad 1: /DMA Peripheral Interface/DMA Peripheral Interface Module/DMA_INT_W -> /IO_CMD
- U201 pad 6: /DMA Peripheral Interface/DMA Peripheral Interface Module/~{RESB} -> RESB
- U202 pad 3: /DMA Peripheral Interface/DMA Peripheral Interface Module/6502_DMA_~{BUSY} -> /DMA Peripheral Interface/~{BUSY}
- U203 pad 21: /DMA Peripheral Interface/DMA Peripheral Interface Module/DMA_INT_R -> /~{IRQ}
- U509 pad 2: Net-(J601-Pin_10) -> /DMA Peripheral Interface/~{BUSY}
- U509 pad 3: /DMA Peripheral Interface/RRW -> /R~{W}
Other:
- board text removed: "SRAM BOARD"

Commit message: Peripheral io layout done; snapshot of current state before redoing much of the rest of the layout.
Parts:
- removed C1005, C1006: 10u, Capacitor_SMD:C_0402_1005Metric
- removed J1003, J1004: Parallel LCD, Connector_IDC:IDC-Header_2x08_P2.54mm_Vertical_SMD
- removed JP1002, JP1003, JP1004: Jumper_2_Bridged, Jumper:SolderJumper-2_P1.3mm_Bridged2Bar_Pad1.0x1.5mm
- removed RV1002, RV1003, RV1004: 10k, Potentiometer_SMD:Potentiometer_Bourns_TC33X_Vertical
- removed TP104, TP106, TP107: TestPoint, TestPoint:TestPoint_Pad_D1.5mm
- added C217: .01u, Capacitor_SMD:C_0402_1005Metric, F.Cu at (253.3, 109.2)
- added C218: .1u, Capacitor_SMD:C_0402_1005Metric, F.Cu at (253.4, 110.2)
- added C301: 10u, Capacitor_SMD:C_0402_1005Metric, F.Cu at (-205.7, 2.54)
- added C302: 1u, Capacitor_SMD:C_0402_1005Metric, F.Cu at (-205.7, 4.51)
- added C303: .01u, Capacitor_SMD:C_0402_1005Metric, F.Cu at (-205.7, 6.48)
- added C304: 10u, Capacitor_SMD:C_0402_1005Metric, F.Cu at (-205.7, 8.45)
- added C305: .01u, Capacitor_SMD:C_0402_1005Metric, F.Cu at (-205.7, 10.4)
- added C306: .01u, Capacitor_SMD:C_0402_1005Metric, F.Cu at (-205.7, 12.4)
- added C307: .01u, Capacitor_SMD:C_0402_1005Metric, F.Cu at (-205.7, 14.4)
- added C308: .1u, Capacitor_SMD:C_0402_1005Metric, F.Cu at (-205.7, 16.3)
- added C309: 1u, Capacitor_SMD:C_0402_1005Metric, F.Cu at (-202.8, 2.54)
- added C310: .01u, Capacitor_SMD:C_0402_1005Metric, F.Cu at (-202.8, 4.51)
- added C311: .1u, Capacitor_SMD:C_0402_1005Metric, F.Cu at (-202.8, 6.48)
- added C312: .01u, Capacitor_SMD:C_0402_1005Metric, F.Cu at (-202.8, 8.45)
- added C313: .1u, Capacitor_SMD:C_0402_1005Metric, F.Cu at (-202.8, 10.4)
- added C314: .01u, Capacitor_SMD:C_0402_1005Metric, F.Cu at (-202.8, 12.4)
- added C315: .1u, Capacitor_SMD:C_0402_1005Metric, F.Cu at (-202.8, 14.4)
- added C316: 1u, Capacitor_SMD:C_0402_1005Metric, F.Cu at (-202.8, 16.3)
- added C317: .01u, Capacitor_SMD:C_0402_1005Metric, F.Cu at (-200.0, 2.54)
- added C318: .1u, Capacitor_SMD:C_0402_1005Metric, F.Cu at (-200.0, 4.51)
- added C319: .1u, Capacitor_SMD:C_0402_1005Metric, F.Cu at (-200.0, 6.48)
- added C320: .1u, Capacitor_SMD:C_0402_1005Metric, F.Cu at (-200.0, 8.45)
- added C321: 1u, Capacitor_SMD:C_0402_1005Metric, F.Cu at (-200.0, 10.4)
- added C322: .01u, Capacitor_SMD:C_0402_1005Metric, F.Cu at (-200.0, 12.4)
- added C323: .1u, Capacitor_SMD:C_0402_1005Metric, F.Cu at (-200.0, 14.4)
- added C324: .01u, Capacitor_SMD:C_0402_1005Metric, F.Cu at (-200.0, 16.3)
- added C325: .1u, Capacitor_SMD:C_0402_1005Metric, F.Cu at (-197.1, 2.54)
- added C326: .01u, Capacitor_SMD:C_0402_1005Metric, F.Cu at (-197.1, 4.51)
- added C327: .1u, Capacitor_SMD:C_0402_1005Metric, F.Cu at (-197.1, 6.48)
- added C328: .01u, Capacitor_SMD:C_0402_1005Metric, F.Cu at (-197.1, 8.45)
- added C329: .1u, Capacitor_SMD:C_0402_1005Metric, F.Cu at (-197.1, 10.4)
- added D301: LED, LED_SMD:LED_0402_1005Metric, F.Cu at (-178.8, -26.6)
- added D302: BAT54CDW, Package_TO_SOT_SMD:SOT-363_SC-70-6, F.Cu at (-193.6, 3.56)
- added D303: BAT54CDW, Package_TO_SOT_SMD:SOT-363_SC-70-6, F.Cu at (-193.6, 7.48)
- added D304: BAT54CDW, Package_TO_SOT_SMD:SOT-363_SC-70-6, F.Cu at (-193.6, 11.4)
- added D305: LED, LED_SMD:LED_0402_1005Metric, F.Cu at (-178.8, -24.6)
- added D306: BAT54CDW, Package_TO_SOT_SMD:SOT-363_SC-70-6, F.Cu at (-193.6, 15.3)
- added D307: BAT54CDW, Package_TO_SOT_SMD:SOT-363_SC-70-6, F.Cu at (-189.3, 3.56)
- added D308: BAT54CDW, Package_TO_SOT_SMD:SOT-363_SC-70-6, F.Cu at (-189.3, 7.48)
- added D309: BAT54CDW, Package_TO_SOT_SMD:SOT-363_SC-70-6, F.Cu at (-189.3, 11.4)
- added J303: Conn_02x16_Odd_Even, Connector_PinHeader_2.54mm:PinHeader_2x16_P2.54mm_Vertical_SMD, F.Cu at (-235.5, 0.54)
- added J304: Conn_02x16_Odd_Even, Connector_PinHeader_2.54mm:PinHeader_2x16_P2.54mm_Vertical_SMD, F.Cu at (-222.7, 0.54)
- added J305: Conn_02x08_Counter_Clockwise, Connector_PinHeader_2.54mm:PinHeader_2x08_P2.54mm_Vertical_SMD, F.Cu at (-200.8, -9.63)
- added JP301: Jumper_2_Small_Open, Jumper:SolderJumper-2_P1.3mm_Open_Pad1.0x1.5mm, F.Cu at (-182.7, -25.8)
- added R309: 33, Resistor_SMD:R_0402_1005Metric, F.Cu at (-192.9, -19.8)
- added R310: 33, Resistor_SMD:R_0402_1005Metric, F.Cu at (-192.9, -17.8)
- added R311: 33, Resistor_SMD:R_0402_1005Metric, F.Cu at (-192.9, -15.8)
- added R312: 33, Resistor_SMD:R_0402_1005Metric, F.Cu at (-192.9, -13.8)
- added R313: 33, Resistor_SMD:R_0402_1005Metric, F.Cu at (-192.9, -11.9)
- added R314: 33, Resistor_SMD:R_0402_1005Metric, F.Cu at (-192.9, -9.87)
- added R315: 33, Resistor_SMD:R_0402_1005Metric, F.Cu at (-192.9, -7.88)
- added R316: 33, Resistor_SMD:R_0402_1005Metric, F.Cu at (-192.9, -5.89)
- added R317: 470, Resistor_SMD:R_0402_1005Metric, F.Cu at (-192.9, -3.90)
- added R318: 100, Resistor_SMD:R_0402_1005Metric, F.Cu at (-190.0, -19.8)
- added R319: 100, Resistor_SMD:R_0402_1005Metric, F.Cu at (-190.0, -17.8)
- added R320: 100, Resistor_SMD:R_0402_1005Metric, F.Cu at (-190.0, -15.8)
- added R321: 100, Resistor_SMD:R_0402_1005Metric, F.Cu at (-190.0, -13.8)
- added R322: 100, Resistor_SMD:R_0402_1005Metric, F.Cu at (-190.0, -11.9)
- added R323: 100, Resistor_SMD:R_0402_1005Metric, F.Cu at (-190.0, -9.87)
- added R324: 100, Resistor_SMD:R_0402_1005Metric, F.Cu at (-190.0, -7.88)
- added R325: 100, Resistor_SMD:R_0402_1005Metric, F.Cu at (-190.0, -5.89)
- added R326: 10K, Resistor_SMD:R_0402_1005Metric, F.Cu at (-190.0, -3.90)
- added R327: 100, Resistor_SMD:R_0402_1005Metric, F.Cu at (-187.1, -19.8)
- added R328: 100, Resistor_SMD:R_0402_1005Metric, F.Cu at (-187.1, -17.8)
- added R329: 100, Resistor_SMD:R_0402_1005Metric, F.Cu at (-187.1, -15.8)
- added R330: 100, Resistor_SMD:R_0402_1005Metric, F.Cu at (-187.1, -13.8)
- added R331: 100, Resistor_SMD:R_0402_1005Metric, F.Cu at (-187.1, -11.9)
- added R332: 100, Resistor_SMD:R_0402_1005Metric, F.Cu at (-187.1, -9.87)
- added R333: 100, Resistor_SMD:R_0402_1005Metric, F.Cu at (-187.1, -7.88)
- added R334: 100, Resistor_SMD:R_0402_1005Metric, F.Cu at (-187.1, -5.89)
- added R335: 100, Resistor_SMD:R_0402_1005Metric, F.Cu at (-187.1, -3.90)
- added R336: 100, Resistor_SMD:R_0402_1005Metric, F.Cu at (-184.2, -19.8)
- added R337: 100, Resistor_SMD:R_0402_1005Metric, F.Cu at (-184.2, -17.8)
- added R338: 100, Resistor_SMD:R_0402_1005Metric, F.Cu at (-184.2, -15.8)
- added R339: 100, Resistor_SMD:R_0402_1005Metric, F.Cu at (-184.2, -13.8)
- added R340: 100, Resistor_SMD:R_0402_1005Metric, F.Cu at (-184.2, -11.9)
- added R341: 100, Resistor_SMD:R_0402_1005Metric, F.Cu at (-184.2, -9.87)
- added R342: 100, Resistor_SMD:R_0402_1005Metric, F.Cu at (-184.2, -7.88)
- added R343: 470, Resistor_SMD:R_0402_1005Metric, F.Cu at (-184.2, -5.89)
- added R344: 100, Resistor_SMD:R_0402_1005Metric, F.Cu at (-184.2, -3.90)
- added R345: 100, Resistor_SMD:R_0402_1005Metric, F.Cu at (-181.3, -19.8)
- added R346: 100, Resistor_SMD:R_0402_1005Metric, F.Cu at (-181.3, -17.8)
- added R347: 100, Resistor_SMD:R_0402_1005Metric, F.Cu at (-181.3, -15.8)
- added R348: 100, Resistor_SMD:R_0402_1005Metric, F.Cu at (-181.3, -13.8)
- added R349: 100, Resistor_SMD:R_0402_1005Metric, F.Cu at (-181.3, -11.9)
- added R350: 100, Resistor_SMD:R_0402_1005Metric, F.Cu at (-181.3, -9.87)
- added R351: 100, Resistor_SMD:R_0402_1005Metric, F.Cu at (-181.3, -7.88)
- added R352: 10k, Resistor_SMD:R_0402_1005Metric, F.Cu at (-181.3, -5.89)
- added R353: 10k, Resistor_SMD:R_0402_1005Metric, F.Cu at (-181.3, -3.90)
- added R354: 10k, Resistor_SMD:R_0402_1005Metric, F.Cu at (-178.3, -19.8)
- added R355: 10k, Resistor_SMD:R_0402_1005Metric, F.Cu at (-178.3, -17.8)
- added R356: 10k, Resistor_SMD:R_0402_1005Metric, F.Cu at (-178.3, -15.8)
- added R357: 10k, Resistor_SMD:R_0402_1005Metric, F.Cu at (-178.3, -13.8)
- added R358: 10k, Resistor_SMD:R_0402_1005Metric, F.Cu at (-178.3, -11.9)
- added R359: 10k, Resistor_SMD:R_0402_1005Metric, F.Cu at (-178.3, -9.87)
- added R506: 1, Resistor_SMD:R_0402_1005Metric, F.Cu at (255.9, 77.3)
- added R507: 1, Resistor_SMD:R_0402_1005Metric, F.Cu at (249.9, 78.7)
- added U301: TXS0108EPW, Package_SO:TSSOP-20_4.4x6.5mm_P0.65mm, F.Cu at (-211.5, -16.8)
- added U302: ~, Package_SO:TSOP-II-44_10.16x18.41mm_P0.8mm, F.Cu at (-234.8, -30.8)
- added U303: 74FCT521ATSOG8, Package_SO:SOIC-20W_7.5x12.8mm_P1.27mm, F.Cu at (-180.7, 8.86)
- added U304: 74ACT139, Package_SO:TSSOP-16_4.4x5mm_P0.65mm, F.Cu at (-180.1, -37.5)
- added U305: 74LVC244APW, Package_SO:TSSOP-20_4.4x6.5mm_P0.65mm, F.Cu at (-211.5, -8.74)
- added U306: ~, Package_SO:TSOP-II-44_10.16x18.41mm_P0.8mm, F.Cu at (-220.5, -30.8)
- added U307: 74LVC244APW, Package_SO:TSSOP-20_4.4x6.5mm_P0.65mm, F.Cu at (-211.5, -0.69)
- added U308: ~, Package_SO:TSOP-II-44_10.16x18.41mm_P0.8mm, F.Cu at (-206.2, -30.8)
- added U309: 74ACT139, Package_SO:TSSOP-16_4.4x5mm_P0.65mm, F.Cu at (-180.1, -30.9)
- added U310: ~, Package_SO:TSOP-II-44_10.16x18.41mm_P0.8mm, F.Cu at (-192.0, -30.8)
- added U311: 74LVC244APW, Package_SO:TSSOP-20_4.4x6.5mm_P0.65mm, F.Cu at (-211.5, 7.36)
- J1002: value Parallel LCD -> LCD_ENs; footprint Connector_IDC:IDC-Header_2x08_P2.54mm_Vertical_SMD -> Connector_PinHeader_2.54mm:PinHeader_1x05_P2.54mm_Vertical
- J301, J302: footprint Connector_PinHeader_2.54mm:PinHeader_2x16_P2.54mm_Vertical_SMD -> Connector_PinHeader_2.54mm:PinHeader_2x16_P2.54mm_Vertical
- moved J1002 358.6 mm to (269.1, 39.2)
- moved J1001 358.3 mm to (260.4, 49.0)
- moved R505 332.4 mm to (253.5, 76.3), turned to -90 degrees
- moved C523 330.5 mm to (252.5, 76.3), turned to -90 degrees
- moved J501 329.2 mm to (241.6, 72.0)
- moved J202 327.8 mm to (241.3, 91.5), turned to -90 degrees
- moved J201 326.9 mm to (256.3, 124.5), turned to -90 degrees
- moved J210 326.4 mm to (254.2, 115.9)
- moved J203 326.0 mm to (254.2, 92.5)
- moved RV501 325.6 mm to (253.5, 79.8), turned to 90 degrees
- moved J205 324.2 mm to (266.1, 92.5)
- moved J204 319.4 mm to (253.8, 128.1), turned to -90 degrees
- moved J301 319.0 mm to (211.9, 46.2), turned to -90 degrees
- moved J206 299.7 mm to (263.4, 110.0)
- moved R1001 291.5 mm to (244.3, 50.2), turned to 90 degrees
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Connections:
- C503 pad 1: +3V3 -> Net-(C503-Pad1)
- C504 pad 1: +2V8 -> Net-(C504-Pad1)
- J1002 pad 2: +5V -> /Character IO/LCD3_EN
- J1002 pad 3: /Character IO/LCD2_CONTRAST -> /Character IO/LCD2_EN
- J1002 pad 4: /Character IO/LCD_RS -> /Character IO/LCD1_EN
- J1002 pad 5: GND -> /Character IO/LCD0_EN
- J501 pad 1: +5V -> GND
- J501 pad 2: GND -> +5V
- R504 pad 1: +3V3 -> +5V
- RV1001 pad 1: GND -> +5V
- RV1001 pad 3: +5V -> GND
Routing:
- net +5V: track 0.00 -> 142.7 mm, vias 0 -> 73
- net /D0: track 0.00 -> 92.6 mm, vias 0 -> 7
- net SDA: track 0.00 -> 87.7 mm, vias 0 -> 5
- net /D1: track 0.00 -> 83.3 mm, vias 0 -> 7
- net SCL: track 0.00 -> 81.4 mm, vias 0 -> 4
- net /D2: track 0.00 -> 81.3 mm, vias 0 -> 8
- net /D3: track 0.00 -> 77.6 mm, vias 0 -> 8
- net /D4: track 0.00 -> 76.2 mm, vias 0 -> 8
- net MISO: track 0.00 -> 75.5 mm, vias 0 -> 3
- net /DMA Peripheral Interface/DMA Peripheral Interface Module/PIC Peripherals/OC_SS_SD: track 0.00 -> 75.2 mm, vias 0 -> 2
- net PHI2: track 0.00 -> 73.0 mm, vias 0 -> 2
- net /D6: track 0.00 -> 72.4 mm, vias 0 -> 9
- net /D5: track 0.00 -> 72.3 mm, vias 0 -> 8
- net /D7: track 0.00 -> 66.6 mm, vias 0 -> 3
- net /DMA Peripheral Interface/DMA Peripheral Interface Module/AUX_SEL: track 0.00 -> 53.7 mm, vias 0 -> 2
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- added copper zone on F.Cu, net +3V3
- added copper zone on In1.Cu, net +3V3
- added copper zone on F.Cu, net +5V
- added copper zone on In1.Cu, net +5V
- added copper zone on In2.Cu, net +5V
- added copper zone on B.Cu, net GND
- added copper zone on F.Cu, net GND
Other:
- board outline added: 127.6 x 98 mm
- copper layers 2 -> 4
- board text removed: "Peripheral i/o"
