File: kicad_project/Hombrew6502Project/ram_banks.kicad_sch (KiCad schematic)
At the start: 114 parts, among them J301 Conn_02x16_Odd_Even, J302 Conn_02x16_Odd_Even, J303 Conn_02x16_Odd_Even, J304 Conn_02x16_Odd_Even, J305 Conn_02x08_Counter_Clockwise, U301 TXS0108EPW, U303 74FCT521ATSOG8, U304 74ACT139, U305 74LVC244APW, U307 74LVC244APW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

Commit message: Peripheral io layout done; snapshot of current state before redoing much of the rest of the layout.
Parts:
- J301, J302: footprint Connector_PinHeader_2.54mm:PinHeader_2x16_P2.54mm_Vertical_SMD -> Connector_PinHeader_2.54mm:PinHeader_2x16_P2.54mm_Vertical
Changed lines of the file:
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@@
 			)
 		)
-		(property "Footprint" "Connector_PinHeader_2.54mm:PinHeader_2x16_P2.54mm_Vertical_SMD"
+		(property "Footprint" "Connector_PinHeader_2.54mm:PinHeader_2x16_P2.54mm_Vertical"
 			(at 27.94 82.55 0)
 			(effects
@@
 			)
 		)
-		(property "Footprint" "Connector_PinHeader_2.54mm:PinHeader_2x16_P2.54mm_Vertical_SMD"
+		(property "Footprint" "Connector_PinHeader_2.54mm:PinHeader_2x16_P2.54mm_Vertical"
 			(at 27.94 38.1 0)
 			(effects
