File: kicad_project/Homebrew6502Project/peripherals.kicad_sch (KiCad schematic)
At the start: 15 parts, among them J402 Micro_SD_Card, J403 Conn_02x03_Odd_Even, U401 74HCT125D, U402 M95512-Axxx-MF

Commit message: Layout of Rev a is finished
Parts:
- J403: now not fitted
Changed lines of the file:
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@@
 		(in_bom yes)
 		(on_board yes)
-		(dnp no)
+		(dnp yes)
 		(fields_autoplaced yes)
 		(property "Reference" "J403"
