File: kicad_project/RamBanks/RamBanks.kicad_sch (KiCad schematic)
At the start: 114 parts, among them J301 Conn_02x16_Odd_Even, J302 Conn_02x16_Odd_Even, J303 Conn_02x16_Odd_Even, J304 Conn_02x16_Odd_Even, J305 Conn_02x08_Counter_Clockwise, U301 TXS0108EPW, U303 74FCT521ATSOG8, U304 74ACT139, U305 74LVC244APW, U307 74LVC244APW, U309 74ACT139, U311 74LVC244APW

Commit message: footprint assignments and separate project for RAM board
Parts:
- removed J301, J302: Conn_02x16_Odd_Even, Connector_PinHeader_2.54mm:PinHeader_2x16_P2.54mm_Vertical_SMD, symbol Connector_Generic:Conn_02x16_Odd_Even
- removed R301, R302, R303, R304, R305, R306, R307, R308: 0, Resistor_SMD:R_0402_1005Metric, symbol Device:R
- added J101, J102: Conn_02x16_Odd_Even, Connector_PinHeader_2.54mm:PinHeader_2x16_P2.54mm_Vertical, symbol Connector_Generic:Conn_02x16_Odd_Even
Connections:
- net +2V8: now also J101.1 (Pin_1)
- net +3V3: now also J101.5 (Pin_5), J101.7 (Pin_7)
- net +5V: now also J101.3 (Pin_3)
- net B20: now also J102.18 (Pin_18)
- net B21: now also J102.16 (Pin_16)
- net B22: now also J102.14 (Pin_14)
- net B23: now also J102.12 (Pin_12)
- net B24: now also J102.10 (Pin_10)
- net B25: now also J102.8 (Pin_8)
- net B26: now also J102.6 (Pin_6)
- net B27: now also J102.4 (Pin_4)
- net D0: now also J101.18 (Pin_18)
- net D1: now also J101.16 (Pin_16)
- net D2: now also J101.14 (Pin_14)
- net D3: now also J101.12 (Pin_12)
- net D4: now also J101.10 (Pin_10)
- net D5: now also J101.8 (Pin_8)
- net D6: now also J101.6 (Pin_6)
- net D7: now also J101.4 (Pin_4)
- net GND: now also J101.2 (Pin_2), J101.20 (Pin_20), J101.27 (Pin_27), J101.31 (Pin_31), J101.32 (Pin_32), J101.9 (Pin_9), J102.1 (Pin_1), J102.15 (Pin_15), J102.2 (Pin_2), J102.20 (Pin_20), J102.26 (Pin_26), J102.30 (Pin_30), J102.32 (Pin_32)
- net PA00: now also J102.31 (Pin_31)
- net PA01: now also J102.29 (Pin_29)
- net PA02: now also J102.27 (Pin_27)
- net PA03: now also J102.25 (Pin_25)
- net PA04: now also J102.23 (Pin_23)
- net PA05: now also J102.21 (Pin_21)
- net PA06: now also J102.19 (Pin_19)
- net PA07: now also J102.17 (Pin_17)
- net PA08: now also J102.13 (Pin_13)
- net PA09: now also J102.11 (Pin_11)
- net PA10: now also J102.9 (Pin_9)
- net PA11: now also J102.7 (Pin_7)
- net PA12: now also J102.5 (Pin_5)
- net PA13: now also J102.3 (Pin_3)
- net PA14: now also J101.25 (Pin_25)
- net PA15: now also J101.23 (Pin_23)
- net PA16: now also J101.21 (Pin_21)
- net PA17: now also J101.19 (Pin_19)
- net PA18: now also J101.17 (Pin_17)
- net PA19: now also J101.15 (Pin_15)
- net PA20: now also J101.13 (Pin_13)
- net PA21: now also J101.11 (Pin_11)
- net PHI2_5: now also J102.28 (Pin_28)
- net R/~{W}: now also J101.30 (Pin_30)
- net P22a: now reaches J304.22 (Pin_22)
- net P22a: now also J102.22 (Pin_22)
- net P24a: now reaches J304.24 (Pin_24)
- net P24a: now also J102.24 (Pin_24)
- net P22: now reaches J303.22 (Pin_22)
- net P22: now also J101.22 (Pin_22)
- net P24: now reaches J303.24 (Pin_24)
- net P24: now also J101.24 (Pin_24)
- net P26: now reaches J303.26 (Pin_26)
- net P26: now also J101.26 (Pin_26)
- net P28: now reaches J303.28 (Pin_28)
- net P28: now also J101.28 (Pin_28)
- net P29: now reaches J303.29 (Pin_29)
- net P29: now also J101.29 (Pin_29)
- no-connect marks 11 -> 4
Other:
- note removed: "BankSel"
- note removed: "Extra outputs"
- note removed: "VAddr LSB"
- note removed: "Vadr MSb's"
- company: Joseph R. Freeston -> (none)
- title: 65c02 Homebrew -> (none)
- moved on the sheet: C301, C302, C303, C304, C305, C306, C307, C308, C309, C310, C311, C312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

Commit message: Layout of Rev a is finished
Parts:
- removed D305: LED, LED_SMD:LED_0402_1005Metric, symbol Device:LED
- removed J305: Conn_02x08_Counter_Clockwise, Connector_PinHeader_2.54mm:PinHeader_2x08_P2.54mm_Vertical_SMD, symbol Connector_Generic:Conn_02x08_Counter_Clockwise
- removed R343: 470, Resistor_SMD:R_0402_1005Metric, symbol Device:R
- added J103: Conn_02x08_Odd_Even, Connector_PinHeader_2.54mm:PinHeader_2x08_P2.54mm_Vertical_SMD, symbol Connector_Generic:Conn_02x08_Odd_Even
Connections:
- net +3V3: now also C309.1
- net +5V: no longer C309.1
- net A0_PREDEC: no longer D302.2 (A02)
- net A16: now also D304.1 (A01); no longer D304.2 (A02)
- net A17: now also D304.5 (A12); no longer D304.1 (A01)
- net GND: now also J103.1 (Pin_1), J103.11 (Pin_11), J103.13 (Pin_13), J103.15 (Pin_15), J103.3 (Pin_3), J103.5 (Pin_5), J103.7 (Pin_7), J103.9 (Pin_9)
- net RW_3: no longer D304.5 (A12)
- net at R355.2, U303.8 (A3): now also J103.8 (Pin_8)
- net at R356.2, U303.11 (A4): now also J103.10 (Pin_10)
- net at R357.2, U303.13 (A5): now also J103.12 (Pin_12)
- net at R358.2, U303.15 (A6): now also J103.14 (Pin_14)
- net at R359.2, U303.17 (A7): now also J103.16 (Pin_16)
- net at R352.2, U303.2 (A0): now also J103.2 (Pin_2)
- net at R353.2, U303.4 (A1): now also J103.4 (Pin_4)
- net at R354.2, U303.6 (A2): now also J103.6 (Pin_6)
- no-connect marks 4 -> 6
Other:
- note removed: "SRAM Data Overvolt Protection"
- company: (none) -> Joseph Russell Freeston
- title: (none) -> CY7C1041DV33 SRAM Board
